Commit message: refactor: update robot dynamics, increase mass properties, and tune Gazebo friction parameters

File: description/body.xacro (robot description, xacro)
@@ -38,5 +38,5 @@
         <axis xyz="0 -1 0"/>
         <limit lower="-0.785" upper="3.14" effort="10.0" velocity="2.0"/>
-        <dynamics damping="10.0" friction="2.0"/>
+        <dynamics damping="0.5" friction="0.1"/>
     </joint>
     <link name="left_shoulder">
@@ -95,5 +95,5 @@
         <axis xyz="0 -1 0"/>
         <limit lower="0" upper="0.873" effort="5.0" velocity="2.0"/>
-        <dynamics damping="10.0" friction="2.0"/>
+        <dynamics damping="0.5" friction="0.1"/>
     </joint>
     <link name="left_forearm">
@@ -126,5 +126,5 @@
         <axis xyz="0 -1 0"/>
         <limit lower="-0.785" upper="3.14" effort="10.0" velocity="2.0"/>
-        <dynamics damping="10.0" friction="2.0"/>
+        <dynamics damping="0.5" friction="0.1"/>
     </joint>
     <link name="right_shoulder">
@@ -183,5 +183,5 @@
         <axis xyz="0 -1 0"/>
         <limit lower="0" upper="0.873" effort="5.0" velocity="2.0"/>
-        <dynamics damping="10.0" friction="2.0"/>
+        <dynamics damping="0.5" friction="0.1"/>
     </joint>
     <link name="right_forearm">

File: description/gripper.xacro (robot description, xacro)
@@ -38,5 +38,5 @@
         <axis xyz="0 1 0"/>
         <limit lower="-0.785" upper="1.047" effort="1.0" velocity="0.5"/>
-        <dynamics damping="3.0" friction="1.0"/>
+        <dynamics damping="0.2" friction="0.05"/>
     </joint>
     <link name="left_gripper_finger1">
@@ -68,5 +68,5 @@
         <axis xyz="0 1 0"/>
         <limit lower="-1.047" upper="0.785" effort="1.0" velocity="0.5"/>
-        <dynamics damping="3.0" friction="1.0"/>
+        <dynamics damping="0.2" friction="0.05"/>
         <mimic joint="left_gripper_finger1_joint" multiplier="-1"/>
     </joint>
@@ -128,5 +128,5 @@
         <axis xyz="0 1 0"/>
         <limit lower="-0.785" upper="1.047" effort="1.0" velocity="0.5"/>
-        <dynamics damping="3.0" friction="1.0"/>
+        <dynamics damping="0.2" friction="0.05"/>
     </joint>
     <link name="right_gripper_finger1">

File: description/head.xacro (robot description, xacro)
@@ -11,5 +11,5 @@
         <axis xyz="0 0 1"/>
         <limit lower="${-pi/2}" upper="${pi/2}" effort="10.0" velocity="0.5"/>
-        <dynamics damping="100.0" friction="20.0"/>  <!-- Very high to prevent flopping -->
+        <dynamics damping="0.5" friction="0.1"/>
     </joint>
     <!-- Neck Link -->

File: description/robot_core.xacro (robot description, xacro)
@@ -9,5 +9,5 @@
     <xacro:property name="body_width" value="0.13"/>
     <xacro:property name="body_height" value="0.36"/>
-    <xacro:property name="body_mass" value="2.5"/>
+    <xacro:property name="body_mass" value="5.0"/>
     <!-- Shoulder Properties -->
     <xacro:property name="shoulder_radius" value="0.035"/>
@@ -43,5 +43,5 @@
     <xacro:property name="chassis_width" value="0.22"/>
     <xacro:property name="chassis_height" value="0.125"/>
-    <xacro:property name="chassis_mass" value="1.0"/>
+    <xacro:property name="chassis_mass" value="10.0"/>
     <xacro:property name="wheel_radius" value="0.06"/>
     <xacro:property name="wheel_thickness" value="0.055"/>
@@ -111,6 +111,6 @@
             </geometry>
         </collision>
-        <xacro:inertial_box mass="0.5" x="${chassis_length}" y="${chassis_width}" z="${chassis_height}">
-            <origin xyz="0 0 ${(chassis_height/2) + (caster_wheel_offset_z * 2) + 0.005}" rpy="0 0 0"/>
+        <xacro:inertial_box mass="5.0" x="${chassis_length}" y="${chassis_width}" z="${chassis_height}">
+            <origin xyz="0 0 0.02" rpy="0 0 0"/>
         </xacro:inertial_box>
     </link>
@@ -123,5 +123,5 @@
         <origin xyz="0 ${wheel_offset_y} 0" rpy="-${pi/2} 0 0" />
         <axis xyz="0 0 1"/>
-        <dynamics damping="0.01" friction="0.01"/>
+        <dynamics damping="0.0" friction="0.0"/>
     </joint>
     <link name="left_wheel">
@@ -143,8 +143,9 @@
     <gazebo reference="left_wheel">
         <material>Gazebo/Black</material>
-        <mu1 value="1.5"/>
-        <mu2 value="1.5"/>
-        <kp value="100000000.0"/>
-        <kd value="1000.0"/>
+        <mu1 value="20.0"/>
+        <mu2 value="20.0"/>
+        <fdir1 value="1 0 0"/>
+        <kp value="1e12"/>
+        <kd value="1.0"/>
     </gazebo>
     <!-- RIGHT WHEEL LINK -->
@@ -154,5 +155,5 @@
         <origin xyz="0 ${-wheel_offset_y} 0" rpy="${pi/2} 0 0" />
         <axis xyz="0 0 -1"/>
-        <dynamics damping="0.01" friction="0.01"/>
+        <dynamics damping="0.0" friction="0.0"/>
     </joint>
     <link name="right_wheel">
@@ -174,8 +175,9 @@
     <gazebo reference="right_wheel">
         <material>Gazebo/Black</material>
-        <mu1 value="1.5"/>
-        <mu2 value="1.5"/>
-        <kp value="100000000.0"/>
-        <kd value="1000.0"/>
+        <mu1 value="20.0"/>
+        <mu2 value="20.0"/>
+        <fdir1 value="1 0 0"/>
+        <kp value="1e12"/>
+        <kd value="1.0"/>
     </gazebo>
     <!-- FRONT CASTER WHEEL LINK -->
