Commit message: feat(description): update URDF body and arm joint configurations and integrate STL meshes
- Torso & Head: Reconfigured body visual/collision geometry to cylinders, updated center of mass/inertia, and adjusted neck length and head joint Z-offsets
- Forearms & Shoulders: Imported body, head, left/right shoulder, and left/right forearm STL meshes with aligned visual offsets; compensated elbow joint axes for local coordinate frame roll
- Right Gripper: Mirrored wrist offsets/yaw from left arm, calibrated fingers (1, 2, 3), and aligned right-gripper.stl mesh origin to finger pivots using point-set registration
- Properties & Fixes: Reduced upper_arm_length to 0.12m in robot_core.xacro, and fixed XML comment mismatch tags and link name typos in gripper.xacro

File: description/body.xacro (robot description, xacro)
@@ -7,23 +7,69 @@
         <child link="body"/>
         <!-- Position body on top of chassis -->
-        <origin xyz="0 0 0.196" rpy="0 0 0"/>
+        <origin xyz="-0.013 0 0.226" rpy="0 0 0"/>
     </joint>
     <link name="body">
-        <visual>
-            <origin xyz="0 0 ${body_height/2}" rpy="0 0 0"/>
-            <geometry>
-                <box size="${body_length} ${body_width} ${body_height}"/>
-            </geometry>
-            <material name="grey"/>
-        </visual>
-        <collision>
-            <origin xyz="0 0 ${body_height/2}" rpy="0 0 0"/>
-            <geometry>
-                <box size="${body_length} ${body_width} ${body_height}"/>
-            </geometry>
-        </collision>
-        <xacro:inertial_box mass="${body_mass}" x="${body_length}" y="${body_width}" z="${body_height}">
-            <origin xyz="0 0 ${body_height/2}" rpy="0 0 0"/>
-        </xacro:inertial_box>
+        <!-- Pelvis (Bottom cylinder) -->
+        <visual>
+            <origin xyz="0 0 0.06" rpy="0 0 0"/>
+            <geometry>
+                <cylinder radius="${body_length*.3}" length="0.18"/>
+            </geometry>
+            <material name="white"/>
+        </visual>
+        <collision>
+            <origin xyz="0 0 0.06" rpy="0 0 0"/>
+            <geometry>
+                <cylinder radius="${body_length*.3}" length="0.18"/>
+            </geometry>
+        </collision>
+        <!-- Waist (Middle cylinder) -->
+        <visual>
+            <origin xyz="0 0 0.17" rpy="0 0 0"/>
+            <geometry>
+                <cylinder radius="${body_length * 0.2}" length="0.12"/>
+            </geometry>
+            <material name="black"/>
+        </visual>
+        <collision>
+            <origin xyz="0 0 0.17" rpy="0 0 0"/>
+            <geometry>
+                <cylinder radius="${body_length * 0.2}" length="0.12"/>
+            </geometry>
+        </collision>
+        <!-- Chest (Third cylinder) -->
+        <visual>
+            <origin xyz="0 0 0.265" rpy="0 0 0"/>
+            <geometry>
+                <cylinder radius="${body_length*.25}" length="0.091"/>
+            </geometry>
+            <material name="white"/>
+        </visual>
+        <collision>
+            <origin xyz="0 0 0.265" rpy="0 0 0"/>
+            <geometry>
+                <cylinder radius="${body_length*.25}" length="0.091"/>
+            </geometry>
+        </collision>
+        <!-- Shoulder (Cylinder connecting both arms) -->
+        <visual>
+            <origin xyz="0 0 0.335" rpy="${pi/2} 0 0"/>
+            <geometry>
+                <cylinder radius="0.04" length="${(body_width/2 + shoulder_radius + 0.01) * 2}"/>
+            </geometry>
+            <material name="white"/>
+        </visual>
+        <collision>
+            <origin xyz="0 0 0.335" rpy="${pi/2} 0 0"/>
+            <geometry>
+                <cylinder radius="0.04" length="${(body_width/2 + shoulder_radius + 0.01) * 2}"/>
+            </geometry>
+        </collision>
+        <!-- Custom Inertial Property (Composite of the Pelvis, Waist, Chest, and Shoulder cylinders) -->
+        <inertial>
+            <origin xyz="0.0 0.0 0.170963" rpy="0 0 0"/>
+            <mass value="${body_mass}"/>
+            <inertia ixx="0.095110" ixy="0.0" ixz="0.0" iyy="0.085819" iyz="0.0" izz="0.018262"/>
+        </inertial>
     </link>
     <gazebo reference="body">
@@ -35,6 +81,6 @@
         <parent link="body"/>
         <child link="left_shoulder"/>
-        <origin xyz="0 ${body_width/2 + shoulder_radius} ${body_height * 0.944444}" rpy="0 0 0"/>
-        <axis xyz="0 -1 0"/>
+        <origin xyz="0 ${body_width/2 + shoulder_radius+0.035} ${body_height * 0.93}" rpy="0.275 0 0"/>
+        <axis xyz="0 -1 0.265"/>
         <limit lower="-0.785" upper="3.14" effort="10.0" velocity="2.0"/>
         <dynamics damping="0.5" friction="0.1"/>
@@ -61,4 +107,21 @@
         <material>Gazebo/DarkGrey</material>
     </gazebo>
+    <!-- +++++++++++++++++++++++++++++++++++++++++++++++++++++++++++++++++++++++++ -->
+    <!-- Visual-only STL mesh attached to left shoulder -->
+    <joint name="external_left_shoulder_mesh_joint" type="fixed">
+        <parent link="left_shoulder"/>
+        <child link="external_left_shoulder_mesh_link"/>
+        <origin xyz="0 0 0" rpy="${pi/2} ${-pi/128} ${pi/2}"/>
+    </joint>
+    <link name="external_left_shoulder_mesh_link">
+        <visual>
+            <origin xyz="-0.2775 -0.50475 0.013000" rpy="0 0 -0.3"/>
+            <geometry>
+                <mesh filename="package://my_bot/description/meshes/left-shoulder.stl" scale="0.001 0.001 0.001"/>
+            </geometry>
+            <material name="grey"/>
+        </visual>
+    </link>
+    <!-- +++++++++++++++++++++++++++++++++++++++++++++++++++++++++++++++++++++++++ -->
     <!-- Left Upper Arm -->
     <joint name="left_upper_arm_joint" type="fixed">
@@ -93,6 +156,6 @@
         <parent link="left_upper_arm"/>
         <child link="left_forearm"/>
-        <origin xyz="0 0 -${upper_arm_length/2}" rpy="0 0 0"/>
-        <axis xyz="0 -1 0"/>
+        <origin xyz="0 0 -${upper_arm_length/2}" rpy="-0.235 0 0"/>
+        <axis xyz="0 -0.9725 -0.2328"/>
         <limit lower="0" upper="0.873" effort="5.0" velocity="2.0"/>
         <dynamics damping="0.5" friction="0.1"/>
@@ -100,5 +163,5 @@
     <link name="left_forearm">
         <visual>
-            <origin xyz="0 0 -${forearm_length/2}" rpy="0 0 0"/>
+            <origin xyz="0.0055 0 -${forearm_length/2}" rpy="0 -0.085 0"/>
             <geometry>
                 <cylinder radius="${forearm_radius}" length="${forearm_length}"/>
@@ -107,5 +170,5 @@
         </visual>
         <collision>
-            <origin xyz="0 0 -${forearm_length/2}" rpy="0 0 0"/>
+            <origin xyz="0.0055  0 -${forearm_length/2}" rpy="0 -0.085 0"/>
             <geometry>
                 <cylinder radius="${forearm_radius}" length="${forearm_length}"/>
@@ -113,5 +176,5 @@
         </collision>
         <xacro:inertial_cylinder mass="${forearm_mass}" length="${forearm_length}" radius="${forearm_radius}">
-            <origin xyz="0 0 -${forearm_length/2}" rpy="0 0 0"/>
+            <origin xyz="0.0055  0 -${forearm_length/2}" rpy="0 -0.085 0"/>
         </xacro:inertial_cylinder>
     </link>
@@ -120,4 +183,21 @@
         <self_collide>false</self_collide>
     </gazebo>
+    <!-- +++++++++++++++++++++++++++++++++++++++++++++++++++++++++++++++++++++++++ -->
+    <!-- Visual-only STL mesh attached to left forearm  -->
+    <joint name="external_left_forearm_mesh_joint" type="fixed">
+        <parent link="left_forearm"/>
+        <child link="external_left_forearm_mesh_link"/>
+        <origin xyz="0 0 0" rpy="${pi/1.9} ${-pi/96} ${pi/2}"/>
+    </joint>
+    <link name="external_left_forearm_mesh_link">
+        <visual>
+            <origin xyz="-0.2235 -0.4125 0.013" rpy="0 0 -0.175"/>
+            <geometry>
+                <mesh filename="package://my_bot/description/meshes/left-forearm.stl" scale="0.001 0.001 0.001"/>
+            </geometry>
+            <material name="grey"/>
+        </visual>
+    </link>
+    <!-- +++++++++++++++++++++++++++++++++++++++++++++++++++++++++++++++++++++++++ -->
     <!-- RIGHT ARM -->
     <!-- Right Shoulder Pitch Joint -->
@@ -125,6 +205,6 @@
         <parent link="body"/>
         <child link="right_shoulder"/>
-        <origin xyz="0 ${-(body_width/2 + shoulder_radius)} ${body_height * 0.944444}" rpy="0 0 0"/>
-        <axis xyz="0 -1 0"/>
+        <origin xyz="0 ${-(body_width/2 + shoulder_radius+0.035)} ${body_height * 0.93}" rpy="-0.275 0 0"/>
+        <axis xyz="0 -1 -0.265"/>
         <limit lower="-0.785" upper="3.14" effort="10.0" velocity="2.0"/>
         <dynamics damping="0.5" friction="0.1"/>
@@ -151,4 +231,21 @@
         <material>Gazebo/DarkGrey</material>
     </gazebo>
+    <!-- +++++++++++++++++++++++++++++++++++++++++++++++++++++++++++++++++++++++++ -->
+    <!-- Visual-only STL mesh attached to right shoulder -->
+    <joint name="external_right_shoulder_mesh_joint" type="fixed">
+        <parent link="right_shoulder"/>
+        <child link="external_right_shoulder_mesh_link"/>
+        <origin xyz="0 0 0" rpy="${pi/2} ${pi/512} ${-pi/2}"/>
+    </joint>
+    <link name="external_right_shoulder_mesh_link">
+        <visual>
+            <origin xyz="-0.2775 -0.50475 -0.013000" rpy="0 0 -0.3"/>
+            <geometry>
+                <mesh filename="package://my_bot/description/meshes/right-sholder.stl" scale="0.001 0.001 0.001"/>
+            </geometry>
+            <material name="grey"/>
+        </visual>
+    </link>
+    <!-- +++++++++++++++++++++++++++++++++++++++++++++++++++++++++++++++++++++++++ -->
     <!-- Right Upper Arm -->
     <joint name="right_upper_arm_joint" type="fixed">
@@ -183,6 +280,6 @@
         <parent link="right_upper_arm"/>
         <child link="right_forearm"/>
-        <origin xyz="0 0 -${upper_arm_length/2}" rpy="0 0 0"/>
-        <axis xyz="0 -1 0"/>
+        <origin xyz="0 0 -${upper_arm_length/2}" rpy="0.235 0 0"/>
+        <axis xyz="0 -0.9725 0.2328"/>
         <limit lower="0" upper="0.873" effort="5.0" velocity="2.0"/>
         <dynamics damping="0.5" friction="0.1"/>
@@ -190,5 +287,5 @@
     <link name="right_forearm">
         <visual>
-            <origin xyz="0 0 -${forearm_length/2}" rpy="0 0 0"/>
+            <origin xyz="0.0055 0 -${forearm_length/2}" rpy="0 -0.085 0"/>
             <geometry>
                 <cylinder radius="${forearm_radius}" length="${forearm_length}"/>
@@ -210,3 +307,35 @@
         <self_collide>false</self_collide>
     </gazebo>
+     <!-- +++++++++++++++++++++++++++++++++++++++++++++++++++++++++++++++++++++++++ -->
+    <!-- Visual-only STL mesh attached to right forearm -->
+    <joint name="external_right_forearm_mesh_joint" type="fixed">
+        <parent link="right_forearm"/>
+        <child link="external_right_forearm_mesh_link"/>
+        <origin xyz="0 0 0" rpy="${pi/2.1} ${-pi/96} ${-pi/2}"/>
+    </joint>
+    <link name="external_right_forearm_mesh_link">
+        <visual>
+            <origin xyz="-0.2235 -0.4125 -0.013" rpy="0 0 -0.165"/>
+            <geometry>
+                <mesh filename="package://my_bot/description/meshes/right-forearm.stl" scale="0.001 0.001 0.001"/>
+            </geometry>
+            <material name="grey"/>
+        </visual>
+    </link>
+    <!-- +++++++++++++++++++++++++++++++++++++++++++++++++++++++++++++++++++++++++ -->
+    <!-- Visual-only STL mesh attached to body -->
+    <joint name="external_body_mesh_joint" type="fixed">
+        <parent link="body"/>
+        <child link="external_body_mesh_link"/>
+        <origin xyz="0 0 0" rpy="${pi/2} 0 ${pi/2}"/>
+    </joint>
+    <link name="external_body_mesh_link">
+        <visual>
+            <origin xyz="0 -0.226 0.013" rpy="0 0 0"/>
+            <geometry>
+                <mesh filename="package://my_bot/description/meshes/body-stl.stl" scale="0.001 0.001 0.001"/>
+            </geometry>
+            <material name="grey"/>
+        </visual>
+    </link>
 </robot>
