Commit message: feat(description): update URDF body and arm joint configurations and integrate STL meshes
- Torso & Head: Reconfigured body visual/collision geometry to cylinders, updated center of mass/inertia, and adjusted neck length and head joint Z-offsets
- Forearms & Shoulders: Imported body, head, left/right shoulder, and left/right forearm STL meshes with aligned visual offsets; compensated elbow joint axes for local coordinate frame roll
- Right Gripper: Mirrored wrist offsets/yaw from left arm, calibrated fingers (1, 2, 3), and aligned right-gripper.stl mesh origin to finger pivots using point-set registration
- Properties & Fixes: Reduced upper_arm_length to 0.12m in robot_core.xacro, and fixed XML comment mismatch tags and link name typos in gripper.xacro

File: description/gripper.xacro (robot description, xacro)
@@ -7,17 +7,17 @@
         <parent link="left_forearm"/>
         <child link="left_gripper_palm"/>
-        <origin xyz="0 0 -${forearm_length}" rpy="0 0 1.571"/>
+        <origin xyz="0.015 0 -${forearm_length}" rpy="0 0 1.571"/>
     </joint>
     <!-- Left Gripper Palm -->
     <link name="left_gripper_palm">
         <visual>
-            <origin xyz="0 0 -${gripper_palm_length/2}" rpy="0 0 0"/>
+             <!-- <origin xyz="0 .00275 -${gripper_palm_length/2}" rpy="0 0 0"/>
             <geometry>
                 <box size="${gripper_palm_width} ${gripper_palm_height} ${gripper_palm_length}"/>
             </geometry>
-            <material name="dark_grey"/>
-        </visual>
-        <collision>
-            <origin xyz="0 0 -${gripper_palm_length/2}" rpy="0 0 0"/>
+            <material name="dark_grey"/> -->
+        </visual>
+        <collision>
+            <origin xyz="0 .00275 -${gripper_palm_length/2}" rpy="0 0 0"/>
             <geometry>
                 <box size="${gripper_palm_width} ${gripper_palm_height} ${gripper_palm_length}"/>
@@ -25,5 +25,5 @@
         </collision>
         <xacro:inertial_box mass="${gripper_palm_mass}" x="${gripper_palm_width}" y="${gripper_palm_height}" z="${gripper_palm_length}">
-            <origin xyz="0 0 -${gripper_palm_length/2}" rpy="0 0 0"/>
+            <origin xyz="0 .00275 -${gripper_palm_length/2}" rpy="0 0 0"/>
         </xacro:inertial_box>
     </link>
@@ -31,16 +31,30 @@
         <material>Gazebo/DarkGrey</material>
     </gazebo>
-    <!-- Left Gripper Finger 1 (revolute joint for opening/closing) -->
-    <joint name="left_gripper_finger1_joint" type="revolute">
+    <!-- +++++++++++++++++++++++++++++++++++++++++++++++++++++++++++++++++++++++++ -->
+    <!-- Visual-only STL mesh attached to left gripper palm (linked to finger2 motion) -->
+    <joint name="external_left_gripper_mesh_joint" type="fixed">
+        <parent link="left_gripper_finger2"/>
+        <child link="external_left_gripper_mesh_link"/>
+        <origin xyz="0.0972 0.0578 -0.3265" rpy="1.684 -0.7833 -0.0124"/>
+    </joint>
+    <link name="external_left_gripper_mesh_link">
+        <visual>
+            <origin xyz="0 0 0" rpy="0 0 0"/>
+            <geometry>
+                <mesh filename="package://my_bot/description/meshes/left-gripper.stl" scale="0.001 0.001 0.001"/>
+            </geometry>
+            <material name="dark_grey"/>
+        </visual>
+    </link>
+    <!-- +++++++++++++++++++++++++++++++++++++++++++++++++++++++++++++++++++++++++ -->
+    <!-- Left Gripper Finger 1 (fixed to the palm) -->
+    <joint name="left_gripper_finger1_joint" type="fixed">
         <parent link="left_gripper_palm"/>
         <child link="left_gripper_finger1"/>
-        <origin xyz="${gripper_palm_width/2} 0 -${gripper_palm_length}" rpy="0 0 0"/>
-        <axis xyz="0 1 0"/>
-        <limit lower="-0.785" upper="1.047" effort="1.0" velocity="0.5"/>
-        <dynamics damping="0.2" friction="0.05"/>
+        <origin xyz="${gripper_palm_width/2.1} -0.001 -${gripper_palm_length}" rpy="-.035 0 0"/>
     </joint>
     <link name="left_gripper_finger1">
         <visual>
-            <origin xyz="${gripper_finger_width/2} 0 -${gripper_finger_length/2}" rpy="0 0 0"/>
+            <origin xyz="${gripper_finger_width/2} 0 -${gripper_finger_length/2.5}" rpy="0 0 0"/>
             <geometry>
                 <box size="${gripper_finger_width} ${gripper_finger_height} ${gripper_finger_length}"/>
@@ -61,17 +75,45 @@
         <material>Gazebo/Grey</material>
     </gazebo>
-    <!-- Left Gripper Finger 2 (mimic finger 1) -->
+     <!-- +++++++++++++++++++++++++++++++++++++++++++++++++++++++++++++++++++++++++ -->
+     <!-- Left Gripper Finger 1 extention (fixed to the finger1) -->
+    <joint name="left_gripper_finger1_ext_joint" type="fixed">
+        <parent link="left_gripper_finger1"/>
+        <child link="left_gripper_finger1_ext"/>
+        <origin xyz="${gripper_palm_width/128} 0 -${gripper_palm_length*1.15}" rpy="0 1.04 0"/>
+    </joint>
+    <link name="left_gripper_finger1_ext">
+        <visual>
+            <origin xyz="${gripper_finger_width/2} 0 -${gripper_finger_length/2}" rpy="0 0 0"/>
+            <geometry>
+                <box size="${gripper_finger_ext_width} ${gripper_finger_ext_height} ${gripper_finger_ext_length}"/>
+            </geometry>
+            <material name="light_grey"/>
+        </visual>
+        <collision>
+            <origin xyz="${gripper_finger_ext_width/2} 0 -${gripper_finger_ext_length/2}" rpy="0 0 0"/>
+            <geometry>
+                <box size="${gripper_finger_ext_width} ${gripper_finger_ext_height} ${gripper_finger_ext_length}"/>
+            </geometry>
+        </collision>
+        <xacro:inertial_box mass="${gripper_finger_ext_mass}" x="${gripper_finger_ext_width}" y="${gripper_finger_ext_height}" z="${gripper_finger_ext_length}">
+            <origin xyz="${gripper_finger_ext_width/2} 0 -${gripper_finger_ext_length/2}" rpy="0 0 0"/>
+        </xacro:inertial_box>
+    </link>
+    <gazebo reference="left_gripper_finger1_ext">
+        <material>Gazebo/Grey</material>
+    </gazebo>
+    <!-- +++++++++++++++++++++++++++++++++++++++++++++++++++++++++++++++++++++++++ -->
+    <!-- Left Gripper Finger 2 (revolute, same shape as finger1, mirrored) -->
     <joint name="left_gripper_finger2_joint" type="revolute">
         <parent link="left_gripper_palm"/>
         <child link="left_gripper_finger2"/>
-        <origin xyz="-${gripper_palm_width/2} 0 -${gripper_palm_length}" rpy="0 0 0"/>
-        <axis xyz="0 1 0"/>
+        <origin xyz="-${gripper_palm_width/8} -0.011 -${gripper_palm_length/1.75}" rpy="-.0325 0.925 0"/>
+        <axis xyz="0 -1 0"/>
         <limit lower="-1.047" upper="0.785" effort="1.0" velocity="0.5"/>
         <dynamics damping="0.2" friction="0.05"/>
-        <mimic joint="left_gripper_finger1_joint" multiplier="-1"/>
     </joint>
     <link name="left_gripper_finger2">
         <visual>
-            <origin xyz="-${gripper_finger_width/2} 0 -${gripper_finger_length/2}" rpy="0 0 0"/>
+            <origin xyz="-${gripper_finger_width/2} 0 -${gripper_finger_length/2.5}" rpy="0 0 0"/>
             <geometry>
                 <box size="${gripper_finger_width} ${gripper_finger_height} ${gripper_finger_length}"/>
@@ -92,4 +134,93 @@
         <material>Gazebo/Grey</material>
     </gazebo>
+    <!-- +++++++++++++++++++++++++++++++++++++++++++++++++++++++++++++++++++++++++ -->
+    <!-- Left Gripper Finger 2 extension (fixed to finger2) -->
+    <joint name="left_gripper_finger2_ext_joint" type="fixed">
+        <parent link="left_gripper_finger2"/>
+        <child link="left_gripper_finger2_ext"/>
+        <origin xyz=".01 0 -${gripper_palm_length}" rpy="0 -.965 0"/>
+    </joint>
+    <link name="left_gripper_finger2_ext">
+        <visual>
+            <origin xyz="-${gripper_finger_width/2} 0 -${gripper_finger_length/3.5}" rpy="0 0 0"/>
+            <geometry>
+                <box size="${gripper_finger_ext_width} ${gripper_finger_ext_height} ${gripper_finger_ext_length}"/>
+            </geometry>
+            <material name="light_grey"/>
+        </visual>
+        <collision>
+            <origin xyz="-${gripper_finger_ext_width/2} 0 -${gripper_finger_ext_length/3.5}" rpy="0 0 0"/>
+            <geometry>
+                <box size="${gripper_finger_ext_width} ${gripper_finger_ext_height} ${gripper_finger_ext_length}"/>
+            </geometry>
+        </collision>
+        <xacro:inertial_box mass="${gripper_finger_ext_mass}" x="${gripper_finger_ext_width}" y="${gripper_finger_ext_height}" z="${gripper_finger_ext_length}">
+            <origin xyz="-${gripper_finger_ext_width/2} 0 -${gripper_finger_ext_length/2}" rpy="0 0 0"/>
+        </xacro:inertial_box>
+    </link>
+    <gazebo reference="left_gripper_finger2_ext">
+        <material>Gazebo/Grey</material>
+    </gazebo>
+    <!-- +++++++++++++++++++++++++++++++++++++++++++++++++++++++++++++++++++++++++ -->
+    <!-- Left Gripper Finger 3 (revolute, same shape as finger1, mirrored, offset from finger2) -->
+    <joint name="left_gripper_finger3_joint" type="revolute">
+        <parent link="left_gripper_palm"/>
+        <child link="left_gripper_finger3"/>
+        <origin xyz="-${gripper_palm_width/8} 0.011 -${gripper_palm_length/1.75}" rpy="-.0325 0.925 0"/>
+        <axis xyz="0 -1 0"/>
+        <limit lower="-1.047" upper="0.785" effort="1.0" velocity="0.5"/>
+        <dynamics damping="0.2" friction="0.05"/>
+        <mimic joint="left_gripper_finger2_joint" multiplier="1"/>
+    </joint>
+    <link name="left_gripper_finger3">
+        <visual>
+            <origin xyz="-${gripper_finger_width/2} 0 -${gripper_finger_length/2.5}" rpy="0 0 0"/>
+            <geometry>
+                <box size="${gripper_finger_width} ${gripper_finger_height} ${gripper_finger_length}"/>
+            </geometry>
+            <material name="light_grey"/>
+        </visual>
+        <collision>
+            <origin xyz="-${gripper_finger_width/2} 0 -${gripper_finger_length/2}" rpy="0 0 0"/>
+            <geometry>
+                <box size="${gripper_finger_width} ${gripper_finger_height} ${gripper_finger_length}"/>
+            </geometry>
+        </collision>
+        <xacro:inertial_box mass="${gripper_finger_mass}" x="${gripper_finger_width}" y="${gripper_finger_height}" z="${gripper_finger_length}">
+            <origin xyz="-${gripper_finger_width/2} 0 -${gripper_finger_length/2}" rpy="0 0 0"/>
+        </xacro:inertial_box>
+    </link>
+    <gazebo reference="left_gripper_finger3">
+        <material>Gazebo/Grey</material>
+    </gazebo>
+    <!-- +++++++++++++++++++++++++++++++++++++++++++++++++++++++++++++++++++++++++ -->
+    <!-- Left Gripper Finger 3 extension (fixed to finger3) -->
+    <joint name="left_gripper_finger3_ext_joint" type="fixed">
+        <parent link="left_gripper_finger3"/>
+        <child link="left_gripper_finger3_ext"/>
+        <origin xyz=".01 0 -${gripper_palm_length}" rpy="0 -.965 0"/>
+    </joint>
+    <link name="left_gripper_finger3_ext">
+        <visual>
+            <origin xyz="-${gripper_finger_width/2} 0 -${gripper_finger_length/3.5}" rpy="0 0 0"/>
+            <geometry>
+                <box size="${gripper_finger_ext_width} ${gripper_finger_ext_height} ${gripper_finger_ext_length}"/>
+            </geometry>
+            <material name="light_grey"/>
+        </visual>
+        <collision>
+            <origin xyz="-${gripper_finger_ext_width/2} 0 -${gripper_finger_ext_length/2}" rpy="0 0 0"/>
+            <geometry>
+                <box size="${gripper_finger_ext_width} ${gripper_finger_ext_height} ${gripper_finger_ext_length}"/>
+            </geometry>
+        </collision>
+        <xacro:inertial_box mass="${gripper_finger_ext_mass}" x="${gripper_finger_ext_width}" y="${gripper_finger_ext_height}" z="${gripper_finger_ext_length}">
+            <origin xyz="-${gripper_finger_ext_width/2} 0 -${gripper_finger_ext_length/2}" rpy="0 0 0"/>
+        </xacro:inertial_box>
+    </link>
+    <gazebo reference="left_gripper_finger3_ext">
+        <material>Gazebo/Grey</material>
+    </gazebo>
+    <!-- +++++++++++++++++++++++++++++++++++++++++++++++++++++++++++++++++++++++++ -->
     <!-- RIGHT GRIPPER ASSEMBLY -->
     <!-- Right Gripper Joint -->
@@ -97,14 +228,14 @@
         <parent link="right_forearm"/>
         <child link="right_gripper_palm"/>
-        <origin xyz="0 0 -${forearm_length}" rpy="0 0 1.571"/>
+        <origin xyz="-0.015 0 -${forearm_length}" rpy="0 0 -1.571"/>
     </joint>
     <!-- Right Gripper Palm -->
     <link name="right_gripper_palm">
         <visual>
-            <origin xyz="0 0 -${gripper_palm_length/2}" rpy="0 0 0"/>
+            <!-- <origin xyz="0 0.0275 -${gripper_palm_length/2}" rpy="0 0 0"/>
             <geometry>
                 <box size="${gripper_palm_width} ${gripper_palm_height} ${gripper_palm_length}"/>
             </geometry>
-            <material name="dark_grey"/>
+            <material name="dark_grey"/> -->
         </visual>
         <collision>
@@ -121,16 +252,30 @@
         <material>Gazebo/DarkGrey</material>
     </gazebo>
-    <!-- Right Gripper Finger 1 -->
-    <joint name="right_gripper_finger1_joint" type="revolute">
+    <!-- +++++++++++++++++++++++++++++++++++++++++++++++++++++++++++++++++++++++++ -->
+    <!-- Visual-only STL mesh attached to right gripper palm (linked to finger2 motion) -->
+    <joint name="external_right_gripper_mesh_joint" type="fixed">
+        <parent link="right_gripper_finger2"/>
+        <child link="external_right_gripper_mesh_link"/>
+        <origin xyz="0.0975 -0.0351 -0.3272" rpy="1.457 -0.783 0.021"/>
+    </joint>
+    <link name="external_right_gripper_mesh_link">
+        <visual>
+            <origin xyz="0 0 0" rpy="0 0 0"/>
+            <geometry>
+                <mesh filename="package://my_bot/description/meshes/right-gripper.stl" scale="0.001 0.001 0.001"/>
+            </geometry>
+            <material name="dark_grey"/>
+        </visual>
+    </link>
+    <!-- +++++++++++++++++++++++++++++++++++++++++++++++++++++++++++++++++++++++++ -->
+    <!-- Right Gripper Finger 1 (fixed to the palm) -->
+    <joint name="right_gripper_finger1_joint" type="fixed">
         <parent link="right_gripper_palm"/>
         <child link="right_gripper_finger1"/>
-        <origin xyz="${gripper_palm_width/2} 0 -${gripper_palm_length}" rpy="0 0 0"/>
-        <axis xyz="0 1 0"/>
-        <limit lower="-0.785" upper="1.047" effort="1.0" velocity="0.5"/>
-        <dynamics damping="0.2" friction="0.05"/>
+        <origin xyz="${gripper_palm_width/2.1} 0.031323 -${gripper_palm_length}" rpy=".035 0 0"/>
     </joint>
     <link name="right_gripper_finger1">
         <visual>
-            <origin xyz="${gripper_finger_width/2} 0 -${gripper_finger_length/2}" rpy="0 0 0"/>
+            <origin xyz="${gripper_finger_width/2} 0 -${gripper_finger_length/2.5}" rpy="0 0 0"/>
             <geometry>
                 <box size="${gripper_finger_width} ${gripper_finger_height} ${gripper_finger_length}"/>
@@ -151,17 +296,45 @@
         <material>Gazebo/Grey</material>
     </gazebo>
-    <!-- Right Gripper Finger 2 (mimic finger 1) -->
+     <!-- +++++++++++++++++++++++++++++++++++++++++++++++++++++++++++++++++++++++++ -->
+     <!-- Right Gripper Finger 1 extension (fixed to finger1) -->
+    <joint name="right_gripper_finger1_ext_joint" type="fixed">
+        <parent link="right_gripper_finger1"/>
+        <child link="right_gripper_finger1_ext"/>
+        <origin xyz="${gripper_palm_width/128} 0 -${gripper_palm_length*1.15}" rpy="0 1.04 0"/>
+    </joint>
+    <link name="right_gripper_finger1_ext">
+        <visual>
+            <origin xyz="${gripper_finger_width/2} 0 -${gripper_finger_length/2}" rpy="0 0 0"/>
+            <geometry>
+                <box size="${gripper_finger_ext_width} ${gripper_finger_ext_height} ${gripper_finger_ext_length}"/>
+            </geometry>
+            <material name="light_grey"/>
+        </visual>
+        <collision>
+            <origin xyz="${gripper_finger_ext_width/2} 0 -${gripper_finger_ext_length/2}" rpy="0 0 0"/>
+            <geometry>
+                <box size="${gripper_finger_ext_width} ${gripper_finger_ext_height} ${gripper_finger_ext_length}"/>
+            </geometry>
+        </collision>
+        <xacro:inertial_box mass="${gripper_finger_ext_mass}" x="${gripper_finger_ext_width}" y="${gripper_finger_ext_height}" z="${gripper_finger_ext_length}">
+            <origin xyz="${gripper_finger_ext_width/2} 0 -${gripper_finger_ext_length/2}" rpy="0 0 0"/>
+        </xacro:inertial_box>
+    </link>
+    <gazebo reference="right_gripper_finger1_ext">
+        <material>Gazebo/Grey</material>
+    </gazebo>
+    <!-- +++++++++++++++++++++++++++++++++++++++++++++++++++++++++++++++++++++++++ -->
+    <!-- Right Gripper Finger 2 (revolute, same shape as finger1, mirrored) -->
     <joint name="right_gripper_finger2_joint" type="revolute">
         <parent link="right_gripper_palm"/>
         <child link="right_gripper_finger2"/>
-        <origin xyz="-${gripper_palm_width/2} 0 -${gripper_palm_length}" rpy="0 0 0"/>
-        <axis xyz="0 1 0"/>
+        <origin xyz="-${gripper_palm_width/8} 0.019 -${gripper_palm_length/1.75}" rpy=".0325 0.925 0"/>
+        <axis xyz="0 -1 0"/>
         <limit lower="-1.047" upper="0.785" effort="1.0" velocity="0.5"/>
-        <dynamics damping="3.0" friction="1.0"/>
-        <mimic joint="right_gripper_finger1_joint" multiplier="-1"/>
+        <dynamics damping="0.2" friction="0.05"/>
     </joint>
     <link name="right_gripper_finger2">
         <visual>
-            <origin xyz="-${gripper_finger_width/2} 0 -${gripper_finger_length/2}" rpy="0 0 0"/>
+            <origin xyz="-${gripper_finger_width/2} 0 -${gripper_finger_length/2.5}" rpy="0 0 0"/>
             <geometry>
                 <box size="${gripper_finger_width} ${gripper_finger_height} ${gripper_finger_length}"/>
@@ -182,3 +355,92 @@
         <material>Gazebo/Grey</material>
     </gazebo>
+    <!-- +++++++++++++++++++++++++++++++++++++++++++++++++++++++++++++++++++++++++ -->
+    <!-- Right Gripper Finger 2 extension (fixed to finger2) -->
+    <joint name="right_gripper_finger2_ext_joint" type="fixed">
+        <parent link="right_gripper_finger2"/>
+        <child link="right_gripper_finger2_ext"/>
+        <origin xyz=".01 0 -${gripper_palm_length}" rpy="0 -.965 0"/>
+    </joint>
+    <link name="right_gripper_finger2_ext">
+        <visual>
+            <origin xyz="-${gripper_finger_width/2} 0 -${gripper_finger_length/3.5}" rpy="0 0 0"/>
+            <geometry>
+                <box size="${gripper_finger_ext_width} ${gripper_finger_ext_height} ${gripper_finger_ext_length}"/>
+            </geometry>
+            <material name="light_grey"/>
+        </visual>
+        <collision>
+            <origin xyz="-${gripper_finger_ext_width/2} 0 -${gripper_finger_ext_length/3.5}" rpy="0 0 0"/>
+            <geometry>
+                <box size="${gripper_finger_ext_width} ${gripper_finger_ext_height} ${gripper_finger_ext_length}"/>
+            </geometry>
+        </collision>
+        <xacro:inertial_box mass="${gripper_finger_ext_mass}" x="${gripper_finger_ext_width}" y="${gripper_finger_ext_height}" z="${gripper_finger_ext_length}">
+            <origin xyz="-${gripper_finger_ext_width/2} 0 -${gripper_finger_ext_length/2}" rpy="0 0 0"/>
+        </xacro:inertial_box>
+    </link>
+    <gazebo reference="right_gripper_finger2_ext">
+        <material>Gazebo/Grey</material>
+    </gazebo>
+    <!-- +++++++++++++++++++++++++++++++++++++++++++++++++++++++++++++++++++++++++ -->
+    <!-- Right Gripper Finger 3 (revolute, same shape as finger1, mirrored, offset from finger2) -->
+    <joint name="right_gripper_finger3_joint" type="revolute">
+        <parent link="right_gripper_palm"/>
+        <child link="right_gripper_finger3"/>
+        <origin xyz="-${gripper_palm_width/8} 0.041 -${gripper_palm_length/1.75}" rpy=".0325 0.925 0"/>
+        <axis xyz="0 -1 0"/>
+        <limit lower="-1.047" upper="0.785" effort="1.0" velocity="0.5"/>
+        <dynamics damping="0.2" friction="0.05"/>
+        <mimic joint="right_gripper_finger2_joint" multiplier="1"/>
+    </joint>
+    <link name="right_gripper_finger3">
+        <visual>
+            <origin xyz="-${gripper_finger_width/2} 0 -${gripper_finger_length/2.5}" rpy="0 0 0"/>
+            <geometry>
+                <box size="${gripper_finger_width} ${gripper_finger_height} ${gripper_finger_length}"/>
+            </geometry>
+            <material name="light_grey"/>
+        </visual>
+        <collision>
+            <origin xyz="-${gripper_finger_width/2} 0 -${gripper_finger_length/2}" rpy="0 0 0"/>
+            <geometry>
+                <box size="${gripper_finger_width} ${gripper_finger_height} ${gripper_finger_length}"/>
+            </geometry>
+        </collision>
+        <xacro:inertial_box mass="${gripper_finger_mass}" x="${gripper_finger_width}" y="${gripper_finger_height}" z="${gripper_finger_length}">
+            <origin xyz="-${gripper_finger_width/2} 0 -${gripper_finger_length/2}" rpy="0 0 0"/>
+        </xacro:inertial_box>
+    </link>
+    <gazebo reference="right_gripper_finger3">
+        <material>Gazebo/Grey</material>
+    </gazebo>
+    <!-- +++++++++++++++++++++++++++++++++++++++++++++++++++++++++++++++++++++++++ -->
+    <!-- Right Gripper Finger 3 extension (fixed to finger3) -->
+    <joint name="right_gripper_finger3_ext_joint" type="fixed">
+        <parent link="right_gripper_finger3"/>
+        <child link="right_gripper_finger3_ext"/>
+        <origin xyz=".01 0 -${gripper_palm_length}" rpy="0 -.965 0"/>
+    </joint>
+    <link name="right_gripper_finger3_ext">
+        <visual>
+            <origin xyz="-${gripper_finger_width/2} 0 -${gripper_finger_length/3.5}" rpy="0 0 0"/>
+            <geometry>
+                <box size="${gripper_finger_ext_width} ${gripper_finger_ext_height} ${gripper_finger_ext_length}"/>
+            </geometry>
+            <material name="light_grey"/>
+        </visual>
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
File: description/head.xacro (robot description, xacro)
@@ -63,3 +63,18 @@
         <material>Gazebo/Red</material>
     </gazebo>
+    <!-- Visual-only STL mesh attached to head -->
+    <joint name="external_head_mesh_joint" type="fixed">
+        <parent link="head"/>
+        <child link="external_head_mesh_link"/>
+        <origin xyz="0 0 0" rpy="${pi/2} 0 ${pi/2}"/>
+    </joint>
+    <link name="external_head_mesh_link">
+        <visual>
+            <origin xyz="0 -0.71738562 0" rpy="0 0 0"/>
+            <geometry>
+                <mesh filename="package://my_bot/description/meshes/head-stl.stl" scale="0.001 0.001 0.001"/>
+            </geometry>
+            <material name="grey"/>
+        </visual>
+    </link>
 </robot>
