Commit message: feat(description): update URDF body and arm joint configurations and integrate STL meshes
- Torso & Head: Reconfigured body visual/collision geometry to cylinders, updated center of mass/inertia, and adjusted neck length and head joint Z-offsets
- Forearms & Shoulders: Imported body, head, left/right shoulder, and left/right forearm STL meshes with aligned visual offsets; compensated elbow joint axes for local coordinate frame roll
- Right Gripper: Mirrored wrist offsets/yaw from left arm, calibrated fingers (1, 2, 3), and aligned right-gripper.stl mesh origin to finger pivots using point-set registration
- Properties & Fixes: Reduced upper_arm_length to 0.12m in robot_core.xacro, and fixed XML comment mismatch tags and link name typos in gripper.xacro

File: description/robot_core.xacro (robot description, xacro)
@@ -11,27 +11,31 @@
     <xacro:property name="body_mass" value="5.0"/>
     <!-- Shoulder Properties -->
-    <xacro:property name="shoulder_radius" value="0.035"/>
+    <xacro:property name="shoulder_radius" value="0.025"/>
     <xacro:property name="shoulder_length" value="0.080"/>
     <xacro:property name="shoulder_mass" value="0.3"/>
     <!-- Upper Arm Properties -->
-    <xacro:property name="upper_arm_radius" value="0.025"/>
+    <xacro:property name="upper_arm_radius" value="0.01"/>
     <xacro:property name="upper_arm_length" value="0.12"/>
     <xacro:property name="upper_arm_mass" value="0.2"/>
     <!-- Forearm Properties -->
-    <xacro:property name="forearm_radius" value="0.020"/>
-    <xacro:property name="forearm_length" value="0.13"/>
+    <xacro:property name="forearm_radius" value="0.0115"/>
+    <xacro:property name="forearm_length" value="0.125"/>
     <xacro:property name="forearm_mass" value="0.15"/>
     <!-- Gripper Properties -->
-    <xacro:property name="gripper_palm_length" value="0.03"/>
+    <xacro:property name="gripper_palm_length" value="0.0335"/>
     <xacro:property name="gripper_palm_width" value="0.05"/>
     <xacro:property name="gripper_palm_height" value="0.03"/>
     <xacro:property name="gripper_palm_mass" value="0.05"/>
-    <xacro:property name="gripper_finger_length" value="0.06"/>
-    <xacro:property name="gripper_finger_width" value="0.015"/>
-    <xacro:property name="gripper_finger_height" value="0.01"/>
+    <xacro:property name="gripper_finger_length" value="0.03"/>
+    <xacro:property name="gripper_finger_width" value="0.00375"/>
+    <xacro:property name="gripper_finger_height" value="0.004"/>
     <xacro:property name="gripper_finger_mass" value="0.01"/>
+    <xacro:property name="gripper_finger_ext_length" value="0.0325"/>
+    <xacro:property name="gripper_finger_ext_width" value="0.005025"/>
+    <xacro:property name="gripper_finger_ext_height" value="0.00425"/>
+    <xacro:property name="gripper_finger_ext_mass" value="0.01"/>
     <!-- Head/Neck Properties -->
     <xacro:property name="neck_radius" value="0.025"/>
-    <xacro:property name="neck_length" value="0.01"/>
+    <xacro:property name="neck_length" value="0.05"/>
     <xacro:property name="neck_mass" value="0.1"/>
     <xacro:property name="head_radius" value="0.08"/>
@@ -42,5 +46,5 @@
     <xacro:property name="chassis_length" value="0.228"/>
     <xacro:property name="chassis_width" value="0.22"/>
-    <xacro:property name="chassis_height" value="0.125"/>
+    <xacro:property name="chassis_height" value="0.0925"/>
     <xacro:property name="chassis_mass" value="10.0"/>
     <xacro:property name="wheel_radius" value="0.06"/>

Commit message: added bonic bot logo

File: description/body.xacro (robot description, xacro)
@@ -338,4 +338,11 @@
             <material name="grey"/>
         </visual>
+        <visual>
+            <origin xyz="0 -0.226 0.013" rpy="0 0 0"/>
+            <geometry>
+                <mesh filename="package://my_bot/description/meshes/BonicLogo-stl.stl" scale="0.001 0.001 0.001"/>
+            </geometry>
+            <material name="black"/>
+        </visual>
     </link>
 </robot>

Commit message: changes in description after testing with gazebo

File: description/body.xacro (robot description, xacro)
@@ -70,5 +70,5 @@
             <origin xyz="0.0 0.0 0.170963" rpy="0 0 0"/>
             <mass value="${body_mass}"/>
-            <inertia ixx="0.095110" ixy="0.0" ixz="0.0" iyy="0.085819" iyz="0.0" izz="0.018262"/>
+            <inertia ixx="0.08667" ixy="0.0" ixz="0.0" iyy="0.08667" iyz="0.0" izz="0.06533"/>
         </inertial>
     </link>

File: description/gripper.xacro (robot description, xacro)
@@ -169,6 +169,6 @@
         <origin xyz="-${gripper_palm_width/8} 0.011 -${gripper_palm_length/1.75}" rpy="-.0325 0.925 0"/>
         <axis xyz="0 -1 0"/>
-        <limit lower="-1.047" upper="0.785" effort="1.0" velocity="0.5"/>
-        <dynamics damping="0.2" friction="0.05"/>
+        <limit lower="-1.047" upper="0.785" effort="10.0" velocity="5.0"/>
+        <dynamics damping="0.0" friction="0.0"/>
         <mimic joint="left_gripper_finger2_joint" multiplier="1"/>
     </joint>
@@ -390,6 +390,6 @@
         <origin xyz="-${gripper_palm_width/8} 0.041 -${gripper_palm_length/1.75}" rpy=".0325 0.925 0"/>
         <axis xyz="0 -1 0"/>
-        <limit lower="-1.047" upper="0.785" effort="1.0" velocity="0.5"/>
-        <dynamics damping="0.2" friction="0.05"/>
+        <limit lower="-1.047" upper="0.785" effort="10.0" velocity="5.0"/>
+        <dynamics damping="0.0" friction="0.0"/>
         <mimic joint="right_gripper_finger2_joint" multiplier="1"/>
     </joint>

File: description/ros2_control.xacro (robot description, xacro)
@@ -53,10 +53,10 @@
       </joint>
       <!-- Grippers - Primary fingers -->
-      <joint name="left_gripper_finger1_joint">
+      <joint name="left_gripper_finger2_joint">
         <command_interface name="position"/>
         <state_interface name="position"/>
         <state_interface name="velocity"/>
       </joint>
-      <joint name="right_gripper_finger1_joint">
+      <joint name="right_gripper_finger2_joint">
         <command_interface name="position"/>
         <state_interface name="position"/>
@@ -64,14 +64,14 @@
       </joint>
       <!-- Grippers - Mimic fingers -->
-      <joint name="left_gripper_finger2_joint">
-        <param name="mimic">left_gripper_finger1_joint</param>
-        <param name="multiplier">-1</param>
+      <joint name="left_gripper_finger3_joint">
+        <param name="mimic">left_gripper_finger2_joint</param>
+        <param name="multiplier">1</param>
         <command_interface name="position"/>
         <state_interface name="position"/>
         <state_interface name="velocity"/>
       </joint>
-      <joint name="right_gripper_finger2_joint">
-        <param name="mimic">right_gripper_finger1_joint</param>
-        <param name="multiplier">-1</param>
+      <joint name="right_gripper_finger3_joint">
+        <param name="mimic">right_gripper_finger2_joint</param>
+        <param name="multiplier">1</param>
         <command_interface name="position"/>
         <state_interface name="position"/>
@@ -152,5 +152,5 @@
       </joint>
       <!-- Grippers - Primary fingers -->
-      <joint name="left_gripper_finger1_joint">
+      <joint name="left_gripper_finger2_joint">
         <command_interface name="position"/>
         <param name="min">-0.785</param>  <!-- -45 degrees -->
@@ -159,5 +159,5 @@
         <state_interface name="velocity"/>
       </joint>
-      <joint name="right_gripper_finger1_joint">
+      <joint name="right_gripper_finger2_joint">
         <command_interface name="position"/>
         <param name="min">-0.785</param>  <!-- -45 degrees -->
