Commit message: added all mesh to the corresponding parts

File: description/body.xacro (robot description, xacro)
@@ -108,17 +108,16 @@
     </gazebo>
     <!-- +++++++++++++++++++++++++++++++++++++++++++++++++++++++++++++++++++++++++ -->
-    <!-- Visual-only STL mesh attached to left shoulder -->
+    <!-- Visual-only colored mesh attached to left shoulder (converted from left-shoulder.glb) -->
     <joint name="external_left_shoulder_mesh_joint" type="fixed">
         <parent link="left_shoulder"/>
         <child link="external_left_shoulder_mesh_link"/>
-        <origin xyz="0 0 0" rpy="${pi/2} ${-pi/128} ${pi/2}"/>
+        <origin xyz="0 0 0" rpy="0 0 0"/>
     </joint>
     <link name="external_left_shoulder_mesh_link">
         <visual>
-            <origin xyz="-0.2775 -0.50475 0.013000" rpy="0 0 -0.3"/>
-            <geometry>
-                <mesh filename="package://my_bot/description/meshes/left-shoulder.stl" scale="0.001 0.001 0.001"/>
-            </geometry>
-            <material name="grey"/>
+            <origin xyz="0 -0.06175 .0185" rpy="0 -0.245 -1.5708"/>
+            <geometry>
+                <mesh filename="package://my_bot/description/meshes/left-shoulder.obj"/>
+            </geometry>
         </visual>
     </link>
@@ -184,18 +183,17 @@
     </gazebo>
     <!-- +++++++++++++++++++++++++++++++++++++++++++++++++++++++++++++++++++++++++ -->
-    <!-- Visual-only STL mesh attached to left forearm  -->
+    <!-- Visual-only colored mesh attached to left forearm (converted from left-forearm.glb)-->
     <joint name="external_left_forearm_mesh_joint" type="fixed">
         <parent link="left_forearm"/>
         <child link="external_left_forearm_mesh_link"/>
-        <origin xyz="0 0 0" rpy="${pi/1.9} ${-pi/96} ${pi/2}"/>
+        <origin xyz="0 0 0" rpy="0 0 0"/>
     </joint>
     <link name="external_left_forearm_mesh_link">
         <visual>
-            <origin xyz="-0.2235 -0.4125 0.013" rpy="0 0 -0.175"/>
-            <geometry>
-                <mesh filename="package://my_bot/description/meshes/left-forearm.stl" scale="0.001 0.001 0.001"/>
-            </geometry>
-            <material name="grey"/>
-        </visual>
+            <origin xyz="0.005 -0.0125 -0.00275" rpy=".1 -0.115 1.5708"/>
+            <geometry>
+                <mesh filename="package://my_bot/description/meshes/left-forearm.obj"/>
+            </geometry>
+        </visual>y
     </link>
     <!-- +++++++++++++++++++++++++++++++++++++++++++++++++++++++++++++++++++++++++ -->
@@ -232,17 +230,16 @@
     </gazebo>
     <!-- +++++++++++++++++++++++++++++++++++++++++++++++++++++++++++++++++++++++++ -->
-    <!-- Visual-only STL mesh attached to right shoulder -->
+    <!-- Visual-only colored mesh attached to right shoulder (converted from right-shoulder.glb) -->
     <joint name="external_right_shoulder_mesh_joint" type="fixed">
         <parent link="right_shoulder"/>
         <child link="external_right_shoulder_mesh_link"/>
-        <origin xyz="0 0 0" rpy="${pi/2} ${pi/512} ${-pi/2}"/>
+        <origin xyz="0 0 0" rpy="0 0 0"/>
     </joint>
     <link name="external_right_shoulder_mesh_link">
         <visual>
-            <origin xyz="-0.2775 -0.50475 -0.013000" rpy="0 0 -0.3"/>
-            <geometry>
-                <mesh filename="package://my_bot/description/meshes/right-sholder.stl" scale="0.001 0.001 0.001"/>
-            </geometry>
-            <material name="grey"/>
+            <origin xyz="0 0.06175 .0185" rpy="0 -0.245 1.5708"/>
+            <geometry>
+                <mesh filename="package://my_bot/description/meshes/right-shoulder.obj"/>
+            </geometry>
         </visual>
     </link>
@@ -307,41 +304,32 @@
         <self_collide>false</self_collide>
     </gazebo>
-     <!-- +++++++++++++++++++++++++++++++++++++++++++++++++++++++++++++++++++++++++ -->
-    <!-- Visual-only STL mesh attached to right forearm -->
+    <!-- +++++++++++++++++++++++++++++++++++++++++++++++++++++++++++++++++++++++++ -->
+    <!-- Visual-only colored mesh attached to right forearm (converted from right-forearm.glb) -->
     <joint name="external_right_forearm_mesh_joint" type="fixed">
         <parent link="right_forearm"/>
         <child link="external_right_forearm_mesh_link"/>
-        <origin xyz="0 0 0" rpy="${pi/2.1} ${-pi/96} ${-pi/2}"/>
+        <origin xyz="0 0 0" rpy="0 0 0"/>
     </joint>
     <link name="external_right_forearm_mesh_link">
         <visual>
-            <origin xyz="-0.2235 -0.4125 -0.013" rpy="0 0 -0.165"/>
-            <geometry>
-                <mesh filename="package://my_bot/description/meshes/right-forearm.stl" scale="0.001 0.001 0.001"/>
-            </geometry>
-            <material name="grey"/>
-        </visual>
-    </link>
-    <!-- +++++++++++++++++++++++++++++++++++++++++++++++++++++++++++++++++++++++++ -->
-    <!-- Visual-only STL mesh attached to body -->
+            <origin xyz="0.005 0.0125 -0.00275" rpy="0.1 0.115 1.5708"/>
+            <geometry>
+                <mesh filename="package://my_bot/description/meshes/right-forearm.obj"/>
+            </geometry>
+        </visual>
+    </link>
+    <!-- +++++++++++++++++++++++++++++++++++++++++++++++++++++++++++++++++++++++++ -->
+    <!-- Visual-only colored mesh attached to body (converted from body.glb) -->
     <joint name="external_body_mesh_joint" type="fixed">
         <parent link="body"/>
         <child link="external_body_mesh_link"/>
-        <origin xyz="0 0 0" rpy="${pi/2} 0 ${pi/2}"/>
+        <origin xyz="0 0 0" rpy="0 0 ${pi/2}"/>
     </joint>
     <link name="external_body_mesh_link">
         <visual>
-            <origin xyz="0 -0.226 0.013" rpy="0 0 0"/>
-            <geometry>
-                <mesh filename="package://my_bot/description/meshes/body-stl.stl" scale="0.001 0.001 0.001"/>
-            </geometry>
-            <material name="grey"/>
-        </visual>
-        <visual>
-            <origin xyz="0 -0.226 0.013" rpy="0 0 0"/>
-            <geometry>
-                <mesh filename="package://my_bot/description/meshes/BonicLogo-stl.stl" scale="0.001 0.001 0.001"/>
-            </geometry>
-            <material name="black"/>
+            <origin xyz="0 -0.0125 -0.225" rpy="0 0 0"/>
+            <geometry>
+                <mesh filename="package://my_bot/description/meshes/body.obj"/>
+            </geometry>
         </visual>
     </link>

File: description/gripper.xacro (robot description, xacro)
@@ -32,17 +32,17 @@
     </gazebo>
     <!-- +++++++++++++++++++++++++++++++++++++++++++++++++++++++++++++++++++++++++ -->
-    <!-- Visual-only STL mesh attached to left gripper palm (linked to finger2 motion) -->
+    <!-- Visual-only colored mesh attached to left gripper (converted from left-gripper.glb) -->
     <joint name="external_left_gripper_mesh_joint" type="fixed">
         <parent link="left_gripper_finger2"/>
         <child link="external_left_gripper_mesh_link"/>
-        <origin xyz="0.0972 0.0578 -0.3265" rpy="1.684 -0.7833 -0.0124"/>
+        <origin xyz="0 0 0" rpy="0 0 0"/>
     </joint>
     <link name="external_left_gripper_mesh_link">
         <visual>
-            <origin xyz="0 0 0" rpy="0 0 0"/>
-            <geometry>
-                <mesh filename="package://my_bot/description/meshes/left-gripper.stl" scale="0.001 0.001 0.001"/>
-            </geometry>
-            <material name="dark_grey"/>
+            <origin xyz="-0.105 0.02 0.0875" rpy=".115 -0.95 0"/>
+            <geometry>
+                <mesh filename="package://my_bot/description/meshes/left-gripper.obj"/>
+            </geometry>
+            <material name="grey"/>
         </visual>
     </link>
@@ -115,9 +115,9 @@
     <link name="left_gripper_finger2">
         <visual>
-            <origin xyz="-${gripper_finger_width/2} 0 -${gripper_finger_length/2.5}" rpy="0 0 0"/>
-            <geometry>
-                <box size="${gripper_finger_width} ${gripper_finger_height} ${gripper_finger_length}"/>
-            </geometry>
-            <material name="light_grey"/>
+            <!-- <origin xyz="-${gripper_finger_width/2} 0 -${gripper_finger_length/2.5}" rpy="0 0 0"/>
+            <geometry>
+                <box size="${gripper_finger_width} ${gripper_finger_height} ${gripper_finger_length}"/>
+            </geometry>
+            <material name="light_grey"/> -->
         </visual>
         <collision>
@@ -143,9 +143,9 @@
     <link name="left_gripper_finger2_ext">
         <visual>
-            <origin xyz="-${gripper_finger_width/2} 0 -${gripper_finger_length/3.5}" rpy="0 0 0"/>
-            <geometry>
-                <box size="${gripper_finger_ext_width} ${gripper_finger_ext_height} ${gripper_finger_ext_length}"/>
-            </geometry>
-            <material name="light_grey"/>
+            <!-- <origin xyz="-${gripper_finger_width/2} 0 -${gripper_finger_length/3.5}" rpy="0 0 0"/>
+            <geometry>
+                <box size="${gripper_finger_ext_width} ${gripper_finger_ext_height} ${gripper_finger_ext_length}"/>
+            </geometry>
+            <material name="light_grey"/> -->
         </visual>
         <collision>
@@ -175,9 +175,9 @@
     <link name="left_gripper_finger3">
         <visual>
-            <origin xyz="-${gripper_finger_width/2} 0 -${gripper_finger_length/2.5}" rpy="0 0 0"/>
-            <geometry>
-                <box size="${gripper_finger_width} ${gripper_finger_height} ${gripper_finger_length}"/>
-            </geometry>
-            <material name="light_grey"/>
+            <!-- <origin xyz="-${gripper_finger_width/2} 0 -${gripper_finger_length/2.5}" rpy="0 0 0"/>
+            <geometry>
+                <box size="${gripper_finger_width} ${gripper_finger_height} ${gripper_finger_length}"/>
+            </geometry>
+            <material name="light_grey"/> -->
         </visual>
         <collision>
@@ -203,9 +203,9 @@
     <link name="left_gripper_finger3_ext">
         <visual>
-            <origin xyz="-${gripper_finger_width/2} 0 -${gripper_finger_length/3.5}" rpy="0 0 0"/>
-            <geometry>
-                <box size="${gripper_finger_ext_width} ${gripper_finger_ext_height} ${gripper_finger_ext_length}"/>
-            </geometry>
-            <material name="light_grey"/>
+            <!-- <origin xyz="-${gripper_finger_width/2} 0 -${gripper_finger_length/3.5}" rpy="0 0 0"/>
+            <geometry>
+                <box size="${gripper_finger_ext_width} ${gripper_finger_ext_height} ${gripper_finger_ext_length}"/>
+            </geometry>
+            <material name="light_grey"/> -->
         </visual>
         <collision>
@@ -253,17 +253,17 @@
     </gazebo>
     <!-- +++++++++++++++++++++++++++++++++++++++++++++++++++++++++++++++++++++++++ -->
-    <!-- Visual-only STL mesh attached to right gripper palm (linked to finger2 motion) -->
+    <!-- Visual-only colored mesh attached to right gripper (converted from right-gripper.glb) -->
     <joint name="external_right_gripper_mesh_joint" type="fixed">
         <parent link="right_gripper_finger2"/>
         <child link="external_right_gripper_mesh_link"/>
-        <origin xyz="0.0975 -0.0351 -0.3272" rpy="1.457 -0.783 0.021"/>
+        <origin xyz="0 0 0" rpy="0 0 0"/>
     </joint>
     <link name="external_right_gripper_mesh_link">
         <visual>
-            <origin xyz="0 0 0" rpy="0 0 0"/>
-            <geometry>
-                <mesh filename="package://my_bot/description/meshes/right-gripper.stl" scale="0.001 0.001 0.001"/>
-            </geometry>
-            <material name="dark_grey"/>
+            <origin xyz="-0.105 0 0.0875" rpy=".115 .95 -3.1416"/>
+            <geometry>
+                <mesh filename="package://my_bot/description/meshes/right-gripper.obj"/>
+            </geometry>
+            <material name="grey"/>
         </visual>
     </link>
@@ -336,9 +336,9 @@
     <link name="right_gripper_finger2">
         <visual>
-            <origin xyz="-${gripper_finger_width/2} 0 -${gripper_finger_length/2.5}" rpy="0 0 0"/>
-            <geometry>
-                <box size="${gripper_finger_width} ${gripper_finger_height} ${gripper_finger_length}"/>
-            </geometry>
-            <material name="light_grey"/>
+            <!-- <origin xyz="-${gripper_finger_width/2} 0 -${gripper_finger_length/2.5}" rpy="0 0 0"/>
+            <geometry>
+                <box size="${gripper_finger_width} ${gripper_finger_height} ${gripper_finger_length}"/>
+            </geometry>
+            <material name="light_grey"/> -->
         </visual>
         <collision>
@@ -364,9 +364,9 @@
     <link name="right_gripper_finger2_ext">
         <visual>
-            <origin xyz="-${gripper_finger_width/2} 0 -${gripper_finger_length/3.5}" rpy="0 0 0"/>
-            <geometry>
-                <box size="${gripper_finger_ext_width} ${gripper_finger_ext_height} ${gripper_finger_ext_length}"/>
-            </geometry>
-            <material name="light_grey"/>
+            <!-- <origin xyz="-${gripper_finger_width/2} 0 -${gripper_finger_length/3.5}" rpy="0 0 0"/>
+            <geometry>
+                <box size="${gripper_finger_ext_width} ${gripper_finger_ext_height} ${gripper_finger_ext_length}"/>
+            </geometry>
+            <material name="light_grey"/> -->
         </visual>
         <collision>
@@ -396,9 +396,9 @@
     <link name="right_gripper_finger3">
         <visual>
-            <origin xyz="-${gripper_finger_width/2} 0 -${gripper_finger_length/2.5}" rpy="0 0 0"/>
-            <geometry>
-                <box size="${gripper_finger_width} ${gripper_finger_height} ${gripper_finger_length}"/>
-            </geometry>
-            <material name="light_grey"/>
+            <!-- <origin xyz="-${gripper_finger_width/2} 0 -${gripper_finger_length/2.5}" rpy="0 0 0"/>
+            <geometry>
+                <box size="${gripper_finger_width} ${gripper_finger_height} ${gripper_finger_length}"/>
+            </geometry>
+            <material name="light_grey"/> -->
         </visual>
         <collision>
@@ -424,9 +424,9 @@
     <link name="right_gripper_finger3_ext">
         <visual>
-            <origin xyz="-${gripper_finger_width/2} 0 -${gripper_finger_length/3.5}" rpy="0 0 0"/>
-            <geometry>
-                <box size="${gripper_finger_ext_width} ${gripper_finger_ext_height} ${gripper_finger_ext_length}"/>
-            </geometry>
-            <material name="light_grey"/>
+            <!-- <origin xyz="-${gripper_finger_width/2} 0 -${gripper_finger_length/3.5}" rpy="0 0 0"/>
+            <geometry>
+                <box size="${gripper_finger_ext_width} ${gripper_finger_ext_height} ${gripper_finger_ext_length}"/>
+            </geometry>
+            <material name="light_grey"/> -->
         </visual>
         <collision>

File: description/head.xacro (robot description, xacro)
@@ -44,9 +44,8 @@
     <link name="head">
         <visual>
-            <origin xyz="0 0 0" rpy="0 0 0"/>
+            <!-- <origin xyz="0 0 0" rpy="0 0 0"/>
             <geometry>
                 <sphere radius="${head_radius}"/>
-            </geometry>
-            <material name="grey"/>
+            </geometry> -->
         </visual>
         <collision>
@@ -63,17 +62,16 @@
         <material>Gazebo/Red</material>
     </gazebo>
-    <!-- Visual-only STL mesh attached to head -->
+    <!-- Visual-only colored mesh attached to head (converted from head.glb) -->
     <joint name="external_head_mesh_joint" type="fixed">
         <parent link="head"/>
         <child link="external_head_mesh_link"/>
-        <origin xyz="0 0 0" rpy="${pi/2} 0 ${pi/2}"/>
+        <origin xyz="0 0 0" rpy="0 0 0"/>
     </joint>
     <link name="external_head_mesh_link">
         <visual>
-            <origin xyz="0 -0.71738562 0" rpy="0 0 0"/>
+            <origin xyz="-0.001 0 -0.1225" rpy="0 0 1.5708"/>
             <geometry>
-                <mesh filename="package://my_bot/description/meshes/head-stl.stl" scale="0.001 0.001 0.001"/>
+                <mesh filename="package://my_bot/description/meshes/head.obj"/>
             </geometry>
-            <material name="grey"/>
         </visual>
     </link>

File: description/robot_core.xacro (robot description, xacro)
@@ -132,8 +132,8 @@
     <link name="left_wheel">
         <visual>
-            <geometry>
+            <!-- <geometry>
                 <cylinder radius="${wheel_radius}" length="${wheel_thickness}"/>
             </geometry>
-            <material name="blue"/>
+            <material name="blue"/> -->
         </visual>
         <collision>
@@ -154,4 +154,18 @@
         <kd value="1.0"/>
     </gazebo>
+    <!-- Visual-only colored mesh attached to left wheel (converted from left-wheel.glb) -->
+    <joint name="external_left_wheel_mesh_joint" type="fixed">
+        <parent link="left_wheel"/>
+        <child link="external_left_wheel_mesh_link"/>
+        <origin xyz="0 0 0" rpy="0 0 0"/>
+    </joint>
+    <link name="external_left_wheel_mesh_link">
+        <visual>
+            <origin xyz="0.0 -0.06925 -0.1443" rpy="-${pi/2} -${pi/2} 0"/>
+            <geometry>
+                <mesh filename="package://my_bot/description/meshes/left-wheel.obj"/>
+            </geometry>
+        </visual>
+    </link>
     <!-- RIGHT WHEEL LINK -->
     <joint name="right_wheel_joint" type="continuous">
@@ -165,8 +179,8 @@
     <link name="right_wheel">
         <visual>
-            <geometry>
+            <!-- <geometry>
                 <cylinder radius="${wheel_radius}" length="${wheel_thickness}"/>
             </geometry>
-            <material name="blue"/>
+            <material name="blue"/> -->
         </visual>
         <collision>
@@ -187,4 +201,18 @@
         <kd value="1.0"/>
     </gazebo>
+    <!-- Visual-only colored mesh attached to right wheel (converted from right-wheel.glb) -->
+    <joint name="external_right_wheel_mesh_joint" type="fixed">
+        <parent link="right_wheel"/>
+        <child link="external_right_wheel_mesh_link"/>
+        <origin xyz="0 0 0" rpy="0 0 0"/>
+    </joint>
+    <link name="external_right_wheel_mesh_link">
+        <visual>
+            <origin xyz="0 -0.06925 -0.1443" rpy="-${pi/2} ${pi/2} 0"/>
+            <geometry>
+                <mesh filename="package://my_bot/description/meshes/right-wheel.obj"/>
+            </geometry>
+        </visual>
+    </link>
     <!-- FRONT CASTER WHEEL LINK -->
     <joint name="front_caster_wheel_joint" type="fixed">
@@ -195,8 +223,8 @@
     <link name="front_caster_wheel">
         <visual>
-            <geometry>
+            <!-- <geometry>
                 <sphere radius="${caster_wheel_radius}"/>
             </geometry>
-            <material name="white"/>
+            <material name="white"/> -->
         </visual>
         <collision>
@@ -222,8 +250,8 @@
     <link name="back_caster_wheel">
         <visual>
-            <geometry>
+            <!-- <geometry>
                 <sphere radius="${caster_wheel_radius}"/>
             </geometry>
-            <material name="white"/>
+            <material name="white"/> -->
         </visual>
         <collision>
