Commit message: changes in z cordinates after visual inconsistency in gazebo

File: description/body.xacro (robot description, xacro)
@@ -7,5 +7,5 @@
         <child link="body"/>
         <!-- Position body on top of chassis -->
-        <origin xyz="-0.013 0 0.226" rpy="0 0 0"/>
+        <origin xyz="-0.013 0 ${body_joint_z_rel_chassis}" rpy="0 0 0"/>
     </joint>
     <link name="body">

File: description/gazebo_control.xacro (robot description, xacro)
@@ -5,6 +5,6 @@
             <left_joint>left_wheel_joint</left_joint>
             <right_joint>right_wheel_joint</right_joint>
-            <wheel_separation>0.2895</wheel_separation>
-            <wheel_diameter>0.12</wheel_diameter>
+            <wheel_separation>${wheel_offset_y * 2}</wheel_separation>
+            <wheel_diameter>${wheel_radius * 2}</wheel_diameter>
             <max_wheel_torque>200</max_wheel_torque>
             <max_wheel_acceleration>10.0</max_wheel_acceleration>

File: description/gripper.xacro (robot description, xacro)
@@ -11,11 +11,4 @@
     <!-- Left Gripper Palm -->
     <link name="left_gripper_palm">
-        <visual>
-             <!-- <origin xyz="0 .00275 -${gripper_palm_length/2}" rpy="0 0 0"/>
-            <geometry>
-                <box size="${gripper_palm_width} ${gripper_palm_height} ${gripper_palm_length}"/>
-            </geometry>
-            <material name="dark_grey"/> -->
-        </visual>
         <collision>
             <origin xyz="0 .00275 -${gripper_palm_length/2}" rpy="0 0 0"/>
@@ -114,11 +107,4 @@
     </joint>
     <link name="left_gripper_finger2">
-        <visual>
-            <!-- <origin xyz="-${gripper_finger_width/2} 0 -${gripper_finger_length/2.5}" rpy="0 0 0"/>
-            <geometry>
-                <box size="${gripper_finger_width} ${gripper_finger_height} ${gripper_finger_length}"/>
-            </geometry>
-            <material name="light_grey"/> -->
-        </visual>
         <collision>
             <origin xyz="-${gripper_finger_width/2} 0 -${gripper_finger_length/2}" rpy="0 0 0"/>
@@ -142,11 +128,4 @@
     </joint>
     <link name="left_gripper_finger2_ext">
-        <visual>
-            <!-- <origin xyz="-${gripper_finger_width/2} 0 -${gripper_finger_length/3.5}" rpy="0 0 0"/>
-            <geometry>
-                <box size="${gripper_finger_ext_width} ${gripper_finger_ext_height} ${gripper_finger_ext_length}"/>
-            </geometry>
-            <material name="light_grey"/> -->
-        </visual>
         <collision>
             <origin xyz="-${gripper_finger_ext_width/2} 0 -${gripper_finger_ext_length/3.5}" rpy="0 0 0"/>
@@ -174,11 +153,4 @@
     </joint>
     <link name="left_gripper_finger3">
-        <visual>
-            <!-- <origin xyz="-${gripper_finger_width/2} 0 -${gripper_finger_length/2.5}" rpy="0 0 0"/>
-            <geometry>
-                <box size="${gripper_finger_width} ${gripper_finger_height} ${gripper_finger_length}"/>
-            </geometry>
-            <material name="light_grey"/> -->
-        </visual>
         <collision>
             <origin xyz="-${gripper_finger_width/2} 0 -${gripper_finger_length/2}" rpy="0 0 0"/>
@@ -202,11 +174,4 @@
     </joint>
     <link name="left_gripper_finger3_ext">
-        <visual>
-            <!-- <origin xyz="-${gripper_finger_width/2} 0 -${gripper_finger_length/3.5}" rpy="0 0 0"/>
-            <geometry>
-                <box size="${gripper_finger_ext_width} ${gripper_finger_ext_height} ${gripper_finger_ext_length}"/>
-            </geometry>
-            <material name="light_grey"/> -->
-        </visual>
         <collision>
             <origin xyz="-${gripper_finger_ext_width/2} 0 -${gripper_finger_ext_length/2}" rpy="0 0 0"/>
@@ -232,11 +197,4 @@
     <!-- Right Gripper Palm -->
     <link name="right_gripper_palm">
-        <visual>
-            <!-- <origin xyz="0 0.0275 -${gripper_palm_length/2}" rpy="0 0 0"/>
-            <geometry>
-                <box size="${gripper_palm_width} ${gripper_palm_height} ${gripper_palm_length}"/>
-            </geometry>
-            <material name="dark_grey"/> -->
-        </visual>
         <collision>
             <origin xyz="0 0 -${gripper_palm_length/2}" rpy="0 0 0"/>
@@ -335,11 +293,4 @@
     </joint>
     <link name="right_gripper_finger2">
-        <visual>
-            <!-- <origin xyz="-${gripper_finger_width/2} 0 -${gripper_finger_length/2.5}" rpy="0 0 0"/>
-            <geometry>
-                <box size="${gripper_finger_width} ${gripper_finger_height} ${gripper_finger_length}"/>
-            </geometry>
-            <material name="light_grey"/> -->
-        </visual>
         <collision>
             <origin xyz="-${gripper_finger_width/2} 0 -${gripper_finger_length/2}" rpy="0 0 0"/>
@@ -363,11 +314,4 @@
     </joint>
     <link name="right_gripper_finger2_ext">
-        <visual>
-            <!-- <origin xyz="-${gripper_finger_width/2} 0 -${gripper_finger_length/3.5}" rpy="0 0 0"/>
-            <geometry>
-                <box size="${gripper_finger_ext_width} ${gripper_finger_ext_height} ${gripper_finger_ext_length}"/>
-            </geometry>
-            <material name="light_grey"/> -->
-        </visual>
         <collision>
             <origin xyz="-${gripper_finger_ext_width/2} 0 -${gripper_finger_ext_length/3.5}" rpy="0 0 0"/>
@@ -395,11 +339,4 @@
     </joint>
     <link name="right_gripper_finger3">
-        <visual>
-            <!-- <origin xyz="-${gripper_finger_width/2} 0 -${gripper_finger_length/2.5}" rpy="0 0 0"/>
-            <geometry>
-                <box size="${gripper_finger_width} ${gripper_finger_height} ${gripper_finger_length}"/>
-            </geometry>
-            <material name="light_grey"/> -->
-        </visual>
         <collision>
             <origin xyz="-${gripper_finger_width/2} 0 -${gripper_finger_length/2}" rpy="0 0 0"/>
@@ -423,11 +360,4 @@
     </joint>
     <link name="right_gripper_finger3_ext">
-        <visual>
-            <!-- <origin xyz="-${gripper_finger_width/2} 0 -${gripper_finger_length/3.5}" rpy="0 0 0"/>
-            <geometry>
-                <box size="${gripper_finger_ext_width} ${gripper_finger_ext_height} ${gripper_finger_ext_length}"/>
-            </geometry>
-            <material name="light_grey"/> -->
-        </visual>
         <collision>
             <origin xyz="-${gripper_finger_ext_width/2} 0 -${gripper_finger_ext_length/2}" rpy="0 0 0"/>

File: description/head.xacro (robot description, xacro)
@@ -43,10 +43,4 @@
     <!-- Head Link -->
     <link name="head">
-        <visual>
-            <!-- <origin xyz="0 0 0" rpy="0 0 0"/>
-            <geometry>
-                <sphere radius="${head_radius}"/>
-            </geometry> -->
-        </visual>
         <collision>
             <origin xyz="0 0 0" rpy="0 0 0"/>

File: description/robot_core.xacro (robot description, xacro)
@@ -59,4 +59,12 @@
     <xacro:property name="caster_wheel_offset_x_back" value="-0.095"/>
     <xacro:property name="caster_wheel_offset_z" value="${wheel_offset_z - wheel_radius + caster_wheel_radius}"/>
+    <!-- Ground clearance & Z-chain parametric definitions -->
+    <xacro:property name="chassis_ground_clearance" value="0.044"/>
+    <xacro:property name="chassis_center_z_rel_chassis" value="${wheel_offset_z - wheel_radius + chassis_ground_clearance + (chassis_height/2)}"/>
+    <xacro:property name="chassis_top_z_rel_chassis" value="${chassis_center_z_rel_chassis + (chassis_height/2)}"/>
+    <xacro:property name="body_ground_gap" value="0.0555"/>
+    <xacro:property name="pelvis_length" value="0.18"/>
+    <xacro:property name="pelvis_z_center" value="0.06"/>
+    <xacro:property name="body_joint_z_rel_chassis" value="${chassis_top_z_rel_chassis + body_ground_gap + (pelvis_length/2 - pelvis_z_center)}"/>
     <material name="white">
         <color rgba="1 1 1 1" />
@@ -92,5 +100,5 @@
         <parent link="base_link"/>
         <child link="base_footprint"/>
-        <origin xyz="0 0 -0.064" rpy="0 0 0"/>
+        <origin xyz="0 0 -${wheel_radius}" rpy="0 0 0"/>
     </joint>
     <link name="base_footprint">
@@ -103,5 +111,5 @@
     <link name="chassis">
         <visual>
-            <origin xyz="0 0 ${(chassis_height/2) + (caster_wheel_offset_z * 2) + 0.005}"/>
+            <origin xyz="0 0 ${chassis_center_z_rel_chassis}"/>
             <geometry>
                 <box size="${chassis_length} ${chassis_width} ${chassis_height}"/>
@@ -110,5 +118,5 @@
         </visual>
         <collision>
-            <origin xyz="0 0 ${(chassis_height/2) + (caster_wheel_offset_z * 2) + 0.005}"/>
+            <origin xyz="0 0 ${chassis_center_z_rel_chassis}"/>
             <geometry>
                 <box size="${chassis_length} ${chassis_width} ${chassis_height}"/>
@@ -122,97 +130,49 @@
         <material>Gazebo/Orange</material>
     </gazebo>
-    <joint name="left_wheel_joint" type="continuous">
-        <parent link="base_link"/>
-        <child link="left_wheel"/>
-        <origin xyz="0 ${wheel_offset_y} 0" rpy="-${pi/2} 0 0" />
-        <axis xyz="0 0 1"/>
-        <limit effort="100.0" velocity="40.0"/>
-        <dynamics damping="0.0" friction="0.0"/>
-    </joint>
-    <link name="left_wheel">
-        <visual>
-            <!-- <geometry>
-                <cylinder radius="${wheel_radius}" length="${wheel_thickness}"/>
-            </geometry>
-            <material name="blue"/> -->
-        </visual>
-        <collision>
-            <geometry>
-                <sphere radius="${wheel_radius}"/>
-            </geometry>
-        </collision>
-        <xacro:inertial_cylinder mass="${wheel_mass}" length="${wheel_thickness}" radius="${wheel_radius}">
+    <!-- WHEEL MACRO -->
+    <xacro:macro name="wheel" params="prefix reflect axis_z mesh_rpy">
+        <joint name="${prefix}_wheel_joint" type="continuous">
+            <parent link="base_link"/>
+            <child link="${prefix}_wheel"/>
+            <origin xyz="0 ${reflect * wheel_offset_y} 0" rpy="${-reflect * pi/2} 0 0" />
+            <axis xyz="0 0 ${axis_z}"/>
+            <limit effort="100.0" velocity="40.0"/>
+            <dynamics damping="0.0" friction="0.0"/>
+        </joint>
+        <link name="${prefix}_wheel">
+            <collision>
+                <geometry>
+                    <sphere radius="${wheel_radius}"/>
+                </geometry>
+            </collision>
+            <xacro:inertial_cylinder mass="${wheel_mass}" length="${wheel_thickness}" radius="${wheel_radius}">
+                <origin xyz="0 0 0" rpy="0 0 0"/>
+            </xacro:inertial_cylinder>
+        </link>
+        <gazebo reference="${prefix}_wheel">
+            <material>Gazebo/Black</material>
+            <mu1 value="10.0"/>
+            <mu2 value="10.0"/>
+            <fdir1 value="1 0 0"/>
+            <kp value="1e7"/>
+            <kd value="1.0"/>
+        </gazebo>
+        <!-- Visual-only colored mesh attached to wheel (converted from ${prefix}-wheel.glb) -->
+        <joint name="external_${prefix}_wheel_mesh_joint" type="fixed">
+            <parent link="${prefix}_wheel"/>
+            <child link="external_${prefix}_wheel_mesh_link"/>
             <origin xyz="0 0 0" rpy="0 0 0"/>
-        </xacro:inertial_cylinder>
-    </link>
-    <gazebo reference="left_wheel">
-        <material>Gazebo/Black</material>
-        <mu1 value="10.0"/>
-        <mu2 value="10.0"/>
-        <fdir1 value="1 0 0"/>
-        <kp value="1e7"/>
-        <kd value="1.0"/>
-    </gazebo>
-    <!-- Visual-only colored mesh attached to left wheel (converted from left-wheel.glb) -->
-    <joint name="external_left_wheel_mesh_joint" type="fixed">
-        <parent link="left_wheel"/>
-        <child link="external_left_wheel_mesh_link"/>
-        <origin xyz="0 0 0" rpy="0 0 0"/>
-    </joint>
-    <link name="external_left_wheel_mesh_link">
-        <visual>
-            <origin xyz="0.0 -0.06925 -0.1443" rpy="-${pi/2} -${pi/2} 0"/>
-            <geometry>
-                <mesh filename="package://my_bot/description/meshes/left-wheel.obj"/>
-            </geometry>
-        </visual>
-    </link>
-    <!-- RIGHT WHEEL LINK -->
-    <joint name="right_wheel_joint" type="continuous">
-        <parent link="base_link"/>
-        <child link="right_wheel"/>
-        <origin xyz="0 ${-wheel_offset_y} 0" rpy="${pi/2} 0 0" />
-        <axis xyz="0 0 -1"/>
-        <limit effort="100.0" velocity="40.0"/>
-        <dynamics damping="0.0" friction="0.0"/>
-    </joint>
-    <link name="right_wheel">
-        <visual>
-            <!-- <geometry>
-                <cylinder radius="${wheel_radius}" length="${wheel_thickness}"/>
-            </geometry>
-            <material name="blue"/> -->
-        </visual>
-        <collision>
-            <geometry>
-                <sphere radius="${wheel_radius}"/>
-            </geometry>
-        </collision>
-        <xacro:inertial_cylinder mass="${wheel_mass}" length="${wheel_thickness}" radius="${wheel_radius}">
-            <origin xyz="0 0 0" rpy="0 0 0"/>
-        </xacro:inertial_cylinder>
-    </link>
-    <gazebo reference="right_wheel">
-        <material>Gazebo/Black</material>
-        <mu1 value="10.0"/>
-        <mu2 value="10.0"/>
-        <fdir1 value="1 0 0"/>
-        <kp value="1e7"/>
-        <kd value="1.0"/>
-    </gazebo>
-    <!-- Visual-only colored mesh attached to right wheel (converted from right-wheel.glb) -->
-    <joint name="external_right_wheel_mesh_joint" type="fixed">
-        <parent link="right_wheel"/>
-        <child link="external_right_wheel_mesh_link"/>
-        <origin xyz="0 0 0" rpy="0 0 0"/>
-    </joint>
-    <link name="external_right_wheel_mesh_link">
-        <visual>
-            <origin xyz="0 -0.06925 -0.1443" rpy="-${pi/2} ${pi/2} 0"/>
-            <geometry>
-                <mesh filename="package://my_bot/description/meshes/right-wheel.obj"/>
-            </geometry>
-        </visual>
-    </link>
+        </joint>
+        <link name="external_${prefix}_wheel_mesh_link">
+            <visual>
+                <origin xyz="0.0 -0.06925 -0.1443" rpy="${mesh_rpy}"/>
+                <geometry>
+                    <mesh filename="package://my_bot/description/meshes/${prefix}-wheel.obj"/>
+                </geometry>
+            </visual>
+        </link>
+    </xacro:macro>
+    <xacro:wheel prefix="left" reflect="1" axis_z="1" mesh_rpy="-${pi/2} -${pi/2} 0"/>
+    <xacro:wheel prefix="right" reflect="-1" axis_z="-1" mesh_rpy="-${pi/2} ${pi/2} 0"/>
     <!-- FRONT CASTER WHEEL LINK -->
     <joint name="front_caster_wheel_joint" type="fixed">
@@ -222,10 +182,4 @@
     </joint>
     <link name="front_caster_wheel">
-        <visual>
-            <!-- <geometry>
-                <sphere radius="${caster_wheel_radius}"/>
-            </geometry>
-            <material name="white"/> -->
-        </visual>
         <collision>
             <geometry>
@@ -241,4 +195,6 @@
         <mu1 value="0.0"/>
         <mu2 value="0.0"/>
+        <kp value="1e7"/>
+        <kd value="1.0"/>
     </gazebo>
     <!-- BACK CASTER WHEEL LINK -->
@@ -249,10 +205,4 @@
     </joint>
     <link name="back_caster_wheel">
-        <visual>
-            <!-- <geometry>
-                <sphere radius="${caster_wheel_radius}"/>
-            </geometry>
-            <material name="white"/> -->
-        </visual>
         <collision>
             <geometry>
@@ -268,4 +218,6 @@
         <mu1 value="0.0"/>
         <mu2 value="0.0"/>
+        <kp value="1e7"/>
+        <kd value="1.0"/>
     </gazebo>
     <!-- ===== IMU Link ===== -->

File: description/ros2_control.xacro (robot description, xacro)
@@ -93,5 +93,5 @@
         <param name="serial_baud">921600</param>
         <param name="encoder_cpr">$(optenv ENCODER_CPR 14040.0)</param>
-        <param name="wheel_radius">0.06</param>   <!-- 0.128m diameter / 2 -->
+        <param name="wheel_radius">${wheel_radius}</param>   <!-- 0.12m diameter / 2 -->
         <param name="max_velocity">10.47</param>   <!-- 100 RPM = 10.47 rad/s -->
       </hardware>
