Commit message: feat: Integrate Extended Kalman Filter (EKF) for robust odometry by fusing wheel and IMU data.

File: description/robot_core.xacro (robot description, xacro)
@@ -231,3 +231,18 @@
         <mu2 value="0.001"/>
     </gazebo>
+    <!-- ===== IMU Link ===== -->
+    <!-- Fixed to base_link — matches frame_id 'imu_link' in sensor_msgs/Imu -->
+    <joint name="imu_joint" type="fixed">
+        <parent link="base_link"/>
+        <child link="imu_link"/>
+        <origin xyz="0 0 0.05" rpy="0 0 0"/>
+    </joint>
+    <link name="imu_link">
+        <visual>
+            <geometry>
+                <box size="0.02 0.02 0.01"/>
+            </geometry>
+            <material name="blue"/>
+        </visual>
+    </link>
 </robot>

Commit message: refactor: adjust caster wheel vertical offset and add damping and friction to wheel joints

File: description/robot_core.xacro (robot description, xacro)
@@ -54,5 +54,5 @@
     <xacro:property name="caster_wheel_offset_x_front" value="0.095"/>
     <xacro:property name="caster_wheel_offset_x_back" value="-0.095"/>
-    <xacro:property name="caster_wheel_offset_z" value="${wheel_offset_z - wheel_radius + caster_wheel_radius + 0.002}"/>
+    <xacro:property name="caster_wheel_offset_z" value="${wheel_offset_z - wheel_radius + caster_wheel_radius}"/>
     <material name="white">
         <color rgba="1 1 1 1" />
@@ -123,4 +123,5 @@
         <origin xyz="0 ${wheel_offset_y} 0" rpy="-${pi/2} 0 0" />
         <axis xyz="0 0 1"/>
+        <dynamics damping="0.01" friction="0.01"/>
     </joint>
     <link name="left_wheel">
@@ -153,4 +154,5 @@
         <origin xyz="0 ${-wheel_offset_y} 0" rpy="${pi/2} 0 0" />
         <axis xyz="0 0 -1"/>
+        <dynamics damping="0.01" friction="0.01"/>
     </joint>
     <link name="right_wheel">

Commit message: chore: increase robot speed limits, update wheel mass, and tune Gazebo friction parameters

File: description/robot_core.xacro (robot description, xacro)
@@ -46,5 +46,5 @@
     <xacro:property name="wheel_radius" value="0.06"/>
     <xacro:property name="wheel_thickness" value="0.055"/>
-    <xacro:property name="wheel_mass" value="0.05"/>
+    <xacro:property name="wheel_mass" value="0.2"/>
     <xacro:property name="wheel_offset_x" value="0.0"/>
     <xacro:property name="wheel_offset_y" value="0.14475"/>
@@ -143,8 +143,8 @@
     <gazebo reference="left_wheel">
         <material>Gazebo/Black</material>
-        <mu1 value="20.0"/>
-        <mu2 value="20.0"/>
+        <mu1 value="2.0"/>
+        <mu2 value="2.0"/>
         <fdir1 value="1 0 0"/>
-        <kp value="1e12"/>
+        <kp value="1e7"/>
         <kd value="1.0"/>
     </gazebo>
@@ -175,8 +175,8 @@
     <gazebo reference="right_wheel">
         <material>Gazebo/Black</material>
-        <mu1 value="20.0"/>
-        <mu2 value="20.0"/>
+        <mu1 value="2.0"/>
+        <mu2 value="2.0"/>
         <fdir1 value="1 0 0"/>
-        <kp value="1e12"/>
+        <kp value="1e7"/>
         <kd value="1.0"/>
     </gazebo>
@@ -205,6 +205,6 @@
     <gazebo reference="front_caster_wheel">
         <material>Gazebo/White</material>
-        <mu1 value="0.001"/>
-        <mu2 value="0.001"/>
+        <mu1 value="0.0"/>
+        <mu2 value="0.0"/>
     </gazebo>
     <!-- BACK CASTER WHEEL LINK -->
@@ -232,6 +232,6 @@
     <gazebo reference="back_caster_wheel">
         <material>Gazebo/White</material>
-        <mu1 value="0.001"/>
-        <mu2 value="0.001"/>
+        <mu1 value="0.0"/>
+        <mu2 value="0.0"/>
     </gazebo>
     <!-- ===== IMU Link ===== -->

File: description/ros2_control.xacro (robot description, xacro)
@@ -9,6 +9,6 @@
       <joint name="left_wheel_joint">
         <command_interface name="velocity">
-          <param name="min">-10</param>
-          <param name="max">10</param>
+          <param name="min">-30</param>
+          <param name="max">30</param>
         </command_interface>
         <state_interface name="position"/>
@@ -17,6 +17,6 @@
       <joint name="right_wheel_joint">
         <command_interface name="velocity">
-          <param name="min">-10</param>
-          <param name="max">10</param>
+          <param name="min">-30</param>
+          <param name="max">30</param>
         </command_interface>
         <state_interface name="position"/>

Commit message: feat: update robot physical properties and add joint limits for improved motion control

File: description/robot_core.xacro (robot description, xacro)
@@ -46,5 +46,5 @@
     <xacro:property name="wheel_radius" value="0.06"/>
     <xacro:property name="wheel_thickness" value="0.055"/>
-    <xacro:property name="wheel_mass" value="0.2"/>
+    <xacro:property name="wheel_mass" value="0.5"/>
     <xacro:property name="wheel_offset_x" value="0.0"/>
     <xacro:property name="wheel_offset_y" value="0.14475"/>
@@ -111,5 +111,5 @@
             </geometry>
         </collision>
-        <xacro:inertial_box mass="5.0" x="${chassis_length}" y="${chassis_width}" z="${chassis_height}">
+        <xacro:inertial_box mass="${chassis_mass}" x="${chassis_length}" y="${chassis_width}" z="${chassis_height}">
             <origin xyz="0 0 0.02" rpy="0 0 0"/>
         </xacro:inertial_box>
@@ -123,4 +123,5 @@
         <origin xyz="0 ${wheel_offset_y} 0" rpy="-${pi/2} 0 0" />
         <axis xyz="0 0 1"/>
+        <limit effort="100.0" velocity="40.0"/>
         <dynamics damping="0.0" friction="0.0"/>
     </joint>
@@ -143,6 +144,6 @@
     <gazebo reference="left_wheel">
         <material>Gazebo/Black</material>
-        <mu1 value="2.0"/>
-        <mu2 value="2.0"/>
+        <mu1 value="0.5"/>
+        <mu2 value="0.8"/>
         <fdir1 value="1 0 0"/>
         <kp value="1e7"/>
@@ -155,4 +156,5 @@
         <origin xyz="0 ${-wheel_offset_y} 0" rpy="${pi/2} 0 0" />
         <axis xyz="0 0 -1"/>
+        <limit effort="100.0" velocity="40.0"/>
         <dynamics damping="0.0" friction="0.0"/>
     </joint>
@@ -175,6 +177,6 @@
     <gazebo reference="right_wheel">
         <material>Gazebo/Black</material>
-        <mu1 value="2.0"/>
-        <mu2 value="2.0"/>
+        <mu1 value="0.5"/>
+        <mu2 value="0.8"/>
         <fdir1 value="1 0 0"/>
         <kp value="1e7"/>

Commit message: feat: add AI agent orchestration and refine navigation configuration settings

File: description/robot_core.xacro (robot description, xacro)
@@ -88,5 +88,5 @@
         <parent link="base_link"/>
         <child link="base_footprint"/>
-        <origin xyz="0 0 0" rpy="0 0 0"/>
+        <origin xyz="0 0 -0.064" rpy="0 0 0"/>
     </joint>
     <link name="base_footprint">
