Commit message: reshaped the camera from square to circle

File: description/camera.xacro (robot description, xacro)
@@ -4,10 +4,11 @@
         <parent link="head"/>
         <child link="camera_link"/>
-        <origin xyz="0.09 0 0.035" rpy="0 0 0"/>
+        <origin xyz="0.0775 0 0.0345" rpy="0 0 0"/>
     </joint>
     <link name="camera_link">
         <visual>
+            <origin xyz="0 0 0" rpy="0 ${pi/2} 0"/>
             <geometry>
-                <box size="0.010 0.03 0.03"/>
+                <cylinder radius="0.005" length="0.005"/>
             </geometry>
             <material name="black"/>

Commit message: fix(description): fix frozen camera stream and adjust sensor mount offsets
camera.xacro:
- Add disableFixedJointLumping on camera_joint and camera_optical_joint
- Add collision and inertial (0.02 kg) to camera_link
- Adjust camera_joint origin to xyz=0.085 0 0.033

lidar.xacro:
- Adjust laser_joint Z offset from 0.145 to 0.18

File: description/camera.xacro (robot description, xacro)
@@ -4,6 +4,13 @@
         <parent link="head"/>
         <child link="camera_link"/>
-        <origin xyz="0.0775 0 0.0345" rpy="0 0 0"/>
+        <origin xyz="0.085 0 0.033" rpy="0 0 0"/>
     </joint>
+    <!-- Prevent URDF→SDF fixed-joint reduction from lumping camera_link
+         into the neck link. Without this, the camera sensor's world pose
+         gets baked at spawn time and never updates when the robot moves,
+         producing a frozen / gray-fill image.  (SDFormat 12 / gz-sim Fortress) -->
+    <gazebo reference="camera_joint">
+        <disableFixedJointLumping>true</disableFixedJointLumping>
+    </gazebo>
     <link name="camera_link">
         <visual>
@@ -14,4 +21,13 @@
             <material name="black"/>
         </visual>
+        <collision>
+            <origin xyz="0 0 0" rpy="0 ${pi/2} 0"/>
+            <geometry>
+                <cylinder radius="0.005" length="0.005"/>
+            </geometry>
+        </collision>
+        <xacro:inertial_cylinder mass="0.02" length="0.005" radius="0.005">
+            <origin xyz="0 0 0" rpy="0 ${pi/2} 0"/>
+        </xacro:inertial_cylinder>
     </link>
     <joint name="camera_optical_joint" type="fixed">
@@ -20,4 +36,8 @@
         <origin xyz="0 0 0" rpy="${-pi/2} 0 ${-pi/2}"/>
     </joint>
+    <!-- Preserve optical frame through URDF→SDF conversion -->
+    <gazebo reference="camera_optical_joint">
+        <disableFixedJointLumping>true</disableFixedJointLumping>
+    </gazebo>
     <link name="camera_link_optical"></link>
     <gazebo reference="camera_link">

File: description/lidar.xacro (robot description, xacro)
@@ -5,5 +5,5 @@
         <child link="laser_frame"/>
         <!-- use below for real robot -->
-        <origin xyz="0.103 0 0.145" rpy="0 0 3.14159"/>
+        <origin xyz="0.103 0 0.18" rpy="0 0 3.14159"/>
         <!-- <origin xyz="0.103 0 0.145" rpy="0 0 0"/> -->
     </joint>
