Commit message: refactor: rename camera node, topics, and frames to face_camera for cross-series compatibility

File: src/nav/bonicbot_a2_description/urdf/camera.xacro (robot description, xacro)
@@ -1,17 +1,17 @@
 <?xml version="1.0"?>
 <robot xmlns:xacro="http://www.ros.org/wiki/xacro" >
-    <joint name="camera_joint" type="fixed">
+    <joint name="face_camera_joint" type="fixed">
         <parent link="head"/>
-        <child link="camera_link"/>
+        <child link="face_camera_link"/>
         <origin xyz="0.085 0 0.033" rpy="0 0 0"/>
     </joint>
-    <!-- Prevent URDF→SDF fixed-joint reduction from lumping camera_link
+    <!-- Prevent URDF→SDF fixed-joint reduction from lumping face_camera_link
          into the neck link. Without this, the camera sensor's world pose
          gets baked at spawn time and never updates when the robot moves,
          producing a frozen / gray-fill image.  (SDFormat 12 / gz-sim Fortress) -->
-    <gazebo reference="camera_joint">
+    <gazebo reference="face_camera_joint">
         <disableFixedJointLumping>true</disableFixedJointLumping>
     </gazebo>
-    <link name="camera_link">
+    <link name="face_camera_link">
         <visual>
             <origin xyz="0 0 0" rpy="0 ${pi/2} 0"/>
@@ -31,17 +31,17 @@
         </xacro:inertial_cylinder>
     </link>
-    <joint name="camera_optical_joint" type="fixed">
-        <parent link="camera_link"/>
-        <child link="camera_link_optical"/>
+    <joint name="face_camera_optical_joint" type="fixed">
+        <parent link="face_camera_link"/>
+        <child link="face_camera_link_optical"/>
         <origin xyz="0 0 0" rpy="${-pi/2} 0 ${-pi/2}"/>
     </joint>
     <!-- Preserve optical frame through URDF→SDF conversion -->
-    <gazebo reference="camera_optical_joint">
+    <gazebo reference="face_camera_optical_joint">
         <disableFixedJointLumping>true</disableFixedJointLumping>
     </gazebo>
-    <link name="camera_link_optical"></link>
-    <gazebo reference="camera_link">
+    <link name="face_camera_link_optical"></link>
+    <gazebo reference="face_camera_link">
         <material>Gazebo/Black</material>
-        <sensor name="camera" type="camera">
+        <sensor name="face_camera" type="camera">
             <pose> 0 0 0 0 0 0 </pose>
             <visualize>true</visualize>
@@ -59,6 +59,6 @@
                 </clip>
             </camera>
-            <topic>/camera/image_raw</topic>
-            <gz_frame_id>camera_link_optical</gz_frame_id>
+            <topic>/face_camera/image_raw</topic>
+            <gz_frame_id>face_camera_link_optical</gz_frame_id>
         </sensor>
     </gazebo>
