Commit message: refactor: reconfigure gripper kinematics by updating joint naming and URDF structures

File: src/nav/bonicbot_a2_description/urdf/gripper.xacro (robot description, xacro)
@@ -27,5 +27,5 @@
     <!-- Visual-only colored mesh attached to left gripper (converted from left-gripper.glb) -->
     <joint name="external_left_gripper_mesh_joint" type="fixed">
-        <parent link="left_gripper_finger2"/>
+        <parent link="left_gripper_finger1"/>
         <child link="external_left_gripper_mesh_link"/>
         <origin xyz="0 0 0" rpy="0 0 0"/>
@@ -42,63 +42,63 @@
     <!-- +++++++++++++++++++++++++++++++++++++++++++++++++++++++++++++++++++++++++ -->
     <!-- Left Gripper Finger 1 (fixed to the palm) -->
-    <joint name="left_gripper_finger1_joint" type="fixed">
+    <joint name="left_gripper_finger3_joint" type="fixed">
+        <parent link="left_gripper_palm"/>
+        <child link="left_gripper_finger3"/>
+        <origin xyz="${gripper_palm_width/2.1} -0.001 -${gripper_palm_length}" rpy="-.035 0 0"/>
+    </joint>
+    <link name="left_gripper_finger3">
+        <visual>
+            <origin xyz="${gripper_finger_width/2} 0 -${gripper_finger_length/2.5}" rpy="0 0 0"/>
+            <geometry>
+                <box size="${gripper_finger_width} ${gripper_finger_height} ${gripper_finger_length}"/>
+            </geometry>
+            <material name="light_grey"/>
+        </visual>
+        <collision>
+            <origin xyz="${gripper_finger_width/2} 0 -${gripper_finger_length/2}" rpy="0 0 0"/>
+            <geometry>
+                <box size="${gripper_finger_width} ${gripper_finger_height} ${gripper_finger_length}"/>
+            </geometry>
+        </collision>
+        <xacro:inertial_box mass="${gripper_finger_mass}" x="${gripper_finger_width}" y="${gripper_finger_height}" z="${gripper_finger_length}">
+            <origin xyz="${gripper_finger_width/2} 0 -${gripper_finger_length/2}" rpy="0 0 0"/>
+        </xacro:inertial_box>
+    </link>
+    <gazebo reference="left_gripper_finger3">
+        <material>Gazebo/Grey</material>
+    </gazebo>
+     <!-- +++++++++++++++++++++++++++++++++++++++++++++++++++++++++++++++++++++++++ -->
+     <!-- Left Gripper Finger 1 extention (fixed to the finger1) -->
+    <joint name="left_gripper_finger3_ext_joint" type="fixed">
+        <parent link="left_gripper_finger3"/>
+        <child link="left_gripper_finger3_ext"/>
+        <origin xyz="${gripper_palm_width/128} 0 -${gripper_palm_length*1.15}" rpy="0 1.04 0"/>
+    </joint>
+    <link name="left_gripper_finger3_ext">
+        <visual>
+            <origin xyz="${gripper_finger_width/2} 0 -${gripper_finger_length/2}" rpy="0 0 0"/>
+            <geometry>
+                <box size="${gripper_finger_ext_width} ${gripper_finger_ext_height} ${gripper_finger_ext_length}"/>
+            </geometry>
+            <material name="light_grey"/>
+        </visual>
+        <collision>
+            <origin xyz="${gripper_finger_ext_width/2} 0 -${gripper_finger_ext_length/2}" rpy="0 0 0"/>
+            <geometry>
+                <box size="${gripper_finger_ext_width} ${gripper_finger_ext_height} ${gripper_finger_ext_length}"/>
+            </geometry>
+        </collision>
+        <xacro:inertial_box mass="${gripper_finger_ext_mass}" x="${gripper_finger_ext_width}" y="${gripper_finger_ext_height}" z="${gripper_finger_ext_length}">
+            <origin xyz="${gripper_finger_ext_width/2} 0 -${gripper_finger_ext_length/2}" rpy="0 0 0"/>
+        </xacro:inertial_box>
+    </link>
+    <gazebo reference="left_gripper_finger3_ext">
+        <material>Gazebo/Grey</material>
+    </gazebo>
+    <!-- +++++++++++++++++++++++++++++++++++++++++++++++++++++++++++++++++++++++++ -->
+    <!-- Left Gripper Finger 2 (revolute, same shape as finger1, mirrored) -->
+    <joint name="left_gripper_finger1_joint" type="revolute">
         <parent link="left_gripper_palm"/>
         <child link="left_gripper_finger1"/>
-        <origin xyz="${gripper_palm_width/2.1} -0.001 -${gripper_palm_length}" rpy="-.035 0 0"/>
-    </joint>
-    <link name="left_gripper_finger1">
-        <visual>
-            <origin xyz="${gripper_finger_width/2} 0 -${gripper_finger_length/2.5}" rpy="0 0 0"/>
-            <geometry>
-                <box size="${gripper_finger_width} ${gripper_finger_height} ${gripper_finger_length}"/>
-            </geometry>
-            <material name="light_grey"/>
-        </visual>
-        <collision>
-            <origin xyz="${gripper_finger_width/2} 0 -${gripper_finger_length/2}" rpy="0 0 0"/>
-            <geometry>
-                <box size="${gripper_finger_width} ${gripper_finger_height} ${gripper_finger_length}"/>
-            </geometry>
-        </collision>
-        <xacro:inertial_box mass="${gripper_finger_mass}" x="${gripper_finger_width}" y="${gripper_finger_height}" z="${gripper_finger_length}">
-            <origin xyz="${gripper_finger_width/2} 0 -${gripper_finger_length/2}" rpy="0 0 0"/>
-        </xacro:inertial_box>
-    </link>
-    <gazebo reference="left_gripper_finger1">
-        <material>Gazebo/Grey</material>
-    </gazebo>
-     <!-- +++++++++++++++++++++++++++++++++++++++++++++++++++++++++++++++++++++++++ -->
-     <!-- Left Gripper Finger 1 extention (fixed to the finger1) -->
-    <joint name="left_gripper_finger1_ext_joint" type="fixed">
-        <parent link="left_gripper_finger1"/>
-        <child link="left_gripper_finger1_ext"/>
-        <origin xyz="${gripper_palm_width/128} 0 -${gripper_palm_length*1.15}" rpy="0 1.04 0"/>
-    </joint>
-    <link name="left_gripper_finger1_ext">
-        <visual>
-            <origin xyz="${gripper_finger_width/2} 0 -${gripper_finger_length/2}" rpy="0 0 0"/>
-            <geometry>
-                <box size="${gripper_finger_ext_width} ${gripper_finger_ext_height} ${gripper_finger_ext_length}"/>
-            </geometry>
-            <material name="light_grey"/>
-        </visual>
-        <collision>
-            <origin xyz="${gripper_finger_ext_width/2} 0 -${gripper_finger_ext_length/2}" rpy="0 0 0"/>
-            <geometry>
-                <box size="${gripper_finger_ext_width} ${gripper_finger_ext_height} ${gripper_finger_ext_length}"/>
-            </geometry>
-        </collision>
-        <xacro:inertial_box mass="${gripper_finger_ext_mass}" x="${gripper_finger_ext_width}" y="${gripper_finger_ext_height}" z="${gripper_finger_ext_length}">
-            <origin xyz="${gripper_finger_ext_width/2} 0 -${gripper_finger_ext_length/2}" rpy="0 0 0"/>
-        </xacro:inertial_box>
-    </link>
-    <gazebo reference="left_gripper_finger1_ext">
-        <material>Gazebo/Grey</material>
-    </gazebo>
-    <!-- +++++++++++++++++++++++++++++++++++++++++++++++++++++++++++++++++++++++++ -->
-    <!-- Left Gripper Finger 2 (revolute, same shape as finger1, mirrored) -->
-    <joint name="left_gripper_finger2_joint" type="revolute">
-        <parent link="left_gripper_palm"/>
-        <child link="left_gripper_finger2"/>
         <origin xyz="-${gripper_palm_width/8} -0.011 -${gripper_palm_length/1.75}" rpy="-.0325 0.925 0"/>
         <axis xyz="0 -1 0"/>
@@ -106,4 +106,50 @@
         <dynamics damping="0.2" friction="0.05"/>
     </joint>
+    <link name="left_gripper_finger1">
+        <collision>
+            <origin xyz="-${gripper_finger_width/2} 0 -${gripper_finger_length/2}" rpy="0 0 0"/>
+            <geometry>
+                <box size="${gripper_finger_width} ${gripper_finger_height} ${gripper_finger_length}"/>
+            </geometry>
+        </collision>
+        <xacro:inertial_box mass="${gripper_finger_mass}" x="${gripper_finger_width}" y="${gripper_finger_height}" z="${gripper_finger_length}">
+            <origin xyz="-${gripper_finger_width/2} 0 -${gripper_finger_length/2}" rpy="0 0 0"/>
+        </xacro:inertial_box>
+    </link>
+    <gazebo reference="left_gripper_finger1">
+        <material>Gazebo/Grey</material>
+    </gazebo>
+    <!-- +++++++++++++++++++++++++++++++++++++++++++++++++++++++++++++++++++++++++ -->
+    <!-- Left Gripper Finger 2 extension (fixed to finger2) -->
+    <joint name="left_gripper_finger1_ext_joint" type="fixed">
+        <parent link="left_gripper_finger1"/>
+        <child link="left_gripper_finger1_ext"/>
+        <origin xyz=".01 0 -${gripper_palm_length}" rpy="0 -.965 0"/>
+    </joint>
+    <link name="left_gripper_finger1_ext">
+        <collision>
+            <origin xyz="-${gripper_finger_ext_width/2} 0 -${gripper_finger_ext_length/3.5}" rpy="0 0 0"/>
+            <geometry>
+                <box size="${gripper_finger_ext_width} ${gripper_finger_ext_height} ${gripper_finger_ext_length}"/>
+            </geometry>
+        </collision>
+        <xacro:inertial_box mass="${gripper_finger_ext_mass}" x="${gripper_finger_ext_width}" y="${gripper_finger_ext_height}" z="${gripper_finger_ext_length}">
+            <origin xyz="-${gripper_finger_ext_width/2} 0 -${gripper_finger_ext_length/2}" rpy="0 0 0"/>
+        </xacro:inertial_box>
+    </link>
+    <gazebo reference="left_gripper_finger1_ext">
+        <material>Gazebo/Grey</material>
+    </gazebo>
+    <!-- +++++++++++++++++++++++++++++++++++++++++++++++++++++++++++++++++++++++++ -->
+    <!-- Left Gripper Finger 3 (revolute, same shape as finger1, mirrored, offset from finger2) -->
+    <joint name="left_gripper_finger2_joint" type="revolute">
+        <parent link="left_gripper_palm"/>
+        <child link="left_gripper_finger2"/>
+        <origin xyz="-${gripper_palm_width/8} 0.011 -${gripper_palm_length/1.75}" rpy="-.0325 0.925 0"/>
+        <axis xyz="0 -1 0"/>
+        <limit lower="-1.047" upper="0.785" effort="10.0" velocity="5.0"/>
+        <dynamics damping="0.0" friction="0.0"/>
+        <mimic joint="left_gripper_finger1_joint" multiplier="1"/>
+    </joint>
     <link name="left_gripper_finger2">
         <collision>
@@ -121,5 +167,5 @@
     </gazebo>
     <!-- +++++++++++++++++++++++++++++++++++++++++++++++++++++++++++++++++++++++++ -->
-    <!-- Left Gripper Finger 2 extension (fixed to finger2) -->
+    <!-- Left Gripper Finger 3 extension (fixed to finger3) -->
     <joint name="left_gripper_finger2_ext_joint" type="fixed">
         <parent link="left_gripper_finger2"/>
@@ -129,5 +175,5 @@
     <link name="left_gripper_finger2_ext">
         <collision>
-            <origin xyz="-${gripper_finger_ext_width/2} 0 -${gripper_finger_ext_length/3.5}" rpy="0 0 0"/>
+            <origin xyz="-${gripper_finger_ext_width/2} 0 -${gripper_finger_ext_length/2}" rpy="0 0 0"/>
             <geometry>
                 <box size="${gripper_finger_ext_width} ${gripper_finger_ext_height} ${gripper_finger_ext_length}"/>
@@ -139,50 +185,4 @@
     </link>
     <gazebo reference="left_gripper_finger2_ext">
-        <material>Gazebo/Grey</material>
-    </gazebo>
-    <!-- +++++++++++++++++++++++++++++++++++++++++++++++++++++++++++++++++++++++++ -->
-    <!-- Left Gripper Finger 3 (revolute, same shape as finger1, mirrored, offset from finger2) -->
-    <joint name="left_gripper_finger3_joint" type="revolute">
-        <parent link="left_gripper_palm"/>
-        <child link="left_gripper_finger3"/>
-        <origin xyz="-${gripper_palm_width/8} 0.011 -${gripper_palm_length/1.75}" rpy="-.0325 0.925 0"/>
-        <axis xyz="0 -1 0"/>
-        <limit lower="-1.047" upper="0.785" effort="10.0" velocity="5.0"/>
-        <dynamics damping="0.0" friction="0.0"/>
-        <mimic joint="left_gripper_finger2_joint" multiplier="1"/>
-    </joint>
-    <link name="left_gripper_finger3">
-        <collision>
-            <origin xyz="-${gripper_finger_width/2} 0 -${gripper_finger_length/2}" rpy="0 0 0"/>
-            <geometry>
-                <box size="${gripper_finger_width} ${gripper_finger_height} ${gripper_finger_length}"/>
-            </geometry>
-        </collision>
-        <xacro:inertial_box mass="${gripper_finger_mass}" x="${gripper_finger_width}" y="${gripper_finger_height}" z="${gripper_finger_length}">
-            <origin xyz="-${gripper_finger_width/2} 0 -${gripper_finger_length/2}" rpy="0 0 0"/>
-        </xacro:inertial_box>
-    </link>
-    <gazebo reference="left_gripper_finger3">
-        <material>Gazebo/Grey</material>
-    </gazebo>
-    <!-- +++++++++++++++++++++++++++++++++++++++++++++++++++++++++++++++++++++++++ -->
-    <!-- Left Gripper Finger 3 extension (fixed to finger3) -->
-    <joint name="left_gripper_finger3_ext_joint" type="fixed">
-        <parent link="left_gripper_finger3"/>
-        <child link="left_gripper_finger3_ext"/>
-        <origin xyz=".01 0 -${gripper_palm_length}" rpy="0 -.965 0"/>
-    </joint>
-    <link name="left_gripper_finger3_ext">
-        <collision>
-            <origin xyz="-${gripper_finger_ext_width/2} 0 -${gripper_finger_ext_length/2}" rpy="0 0 0"/>
-            <geometry>
-                <box size="${gripper_finger_ext_width} ${gripper_finger_ext_height} ${gripper_finger_ext_length}"/>
-            </geometry>
-        </collision>
-        <xacro:inertial_box mass="${gripper_finger_ext_mass}" x="${gripper_finger_ext_width}" y="${gripper_finger_ext_height}" z="${gripper_finger_ext_length}">
-            <origin xyz="-${gripper_finger_ext_width/2} 0 -${gripper_finger_ext_length/2}" rpy="0 0 0"/>
-        </xacro:inertial_box>
-    </link>
-    <gazebo reference="left_gripper_finger3_ext">
         <material>Gazebo/Grey</material>
     </gazebo>
@@ -213,5 +213,5 @@
     <!-- Visual-only colored mesh attached to right gripper (converted from right-gripper.glb) -->
     <joint name="external_right_gripper_mesh_joint" type="fixed">
-        <parent link="right_gripper_finger2"/>
+        <parent link="right_gripper_finger1"/>
         <child link="external_right_gripper_mesh_link"/>
         <origin xyz="0 0 0" rpy="0 0 0"/>
@@ -228,63 +228,63 @@
     <!-- +++++++++++++++++++++++++++++++++++++++++++++++++++++++++++++++++++++++++ -->
     <!-- Right Gripper Finger 1 (fixed to the palm) -->
-    <joint name="right_gripper_finger1_joint" type="fixed">
+    <joint name="right_gripper_finger3_joint" type="fixed">
+        <parent link="right_gripper_palm"/>
+        <child link="right_gripper_finger3"/>
+        <origin xyz="${gripper_palm_width/2.1} 0.031323 -${gripper_palm_length}" rpy=".035 0 0"/>
+    </joint>
+    <link name="right_gripper_finger3">
+        <visual>
+            <origin xyz="${gripper_finger_width/2} 0 -${gripper_finger_length/2.5}" rpy="0 0 0"/>
+            <geometry>
+                <box size="${gripper_finger_width} ${gripper_finger_height} ${gripper_finger_length}"/>
+            </geometry>
+            <material name="light_grey"/>
+        </visual>
+        <collision>
+            <origin xyz="${gripper_finger_width/2} 0 -${gripper_finger_length/2}" rpy="0 0 0"/>
+            <geometry>
+                <box size="${gripper_finger_width} ${gripper_finger_height} ${gripper_finger_length}"/>
+            </geometry>
+        </collision>
+        <xacro:inertial_box mass="${gripper_finger_mass}" x="${gripper_finger_width}" y="${gripper_finger_height}" z="${gripper_finger_length}">
+            <origin xyz="${gripper_finger_width/2} 0 -${gripper_finger_length/2}" rpy="0 0 0"/>
+        </xacro:inertial_box>
+    </link>
+    <gazebo reference="right_gripper_finger3">
+        <material>Gazebo/Grey</material>
+    </gazebo>
+     <!-- +++++++++++++++++++++++++++++++++++++++++++++++++++++++++++++++++++++++++ -->
+     <!-- Right Gripper Finger 1 extension (fixed to finger1) -->
+    <joint name="right_gripper_finger3_ext_joint" type="fixed">
+        <parent link="right_gripper_finger3"/>
+        <child link="right_gripper_finger3_ext"/>
+        <origin xyz="${gripper_palm_width/128} 0 -${gripper_palm_length*1.15}" rpy="0 1.04 0"/>
+    </joint>
+    <link name="right_gripper_finger3_ext">
+        <visual>
+            <origin xyz="${gripper_finger_width/2} 0 -${gripper_finger_length/2}" rpy="0 0 0"/>
+            <geometry>
+                <box size="${gripper_finger_ext_width} ${gripper_finger_ext_height} ${gripper_finger_ext_length}"/>
+            </geometry>
+            <material name="light_grey"/>
+        </visual>
+        <collision>
+            <origin xyz="${gripper_finger_ext_width/2} 0 -${gripper_finger_ext_length/2}" rpy="0 0 0"/>
+            <geometry>
+                <box size="${gripper_finger_ext_width} ${gripper_finger_ext_height} ${gripper_finger_ext_length}"/>
+            </geometry>
+        </collision>
+        <xacro:inertial_box mass="${gripper_finger_ext_mass}" x="${gripper_finger_ext_width}" y="${gripper_finger_ext_height}" z="${gripper_finger_ext_length}">
+            <origin xyz="${gripper_finger_ext_width/2} 0 -${gripper_finger_ext_length/2}" rpy="0 0 0"/>
+        </xacro:inertial_box>
+    </link>
+    <gazebo reference="right_gripper_finger3_ext">
+        <material>Gazebo/Grey</material>
+    </gazebo>
+    <!-- +++++++++++++++++++++++++++++++++++++++++++++++++++++++++++++++++++++++++ -->
+    <!-- Right Gripper Finger 2 (revolute, same shape as finger1, mirrored) -->
+    <joint name="right_gripper_finger1_joint" type="revolute">
         <parent link="right_gripper_palm"/>
         <child link="right_gripper_finger1"/>
-        <origin xyz="${gripper_palm_width/2.1} 0.031323 -${gripper_palm_length}" rpy=".035 0 0"/>
-    </joint>
-    <link name="right_gripper_finger1">
-        <visual>
-            <origin xyz="${gripper_finger_width/2} 0 -${gripper_finger_length/2.5}" rpy="0 0 0"/>
-            <geometry>
-                <box size="${gripper_finger_width} ${gripper_finger_height} ${gripper_finger_length}"/>
-            </geometry>
-            <material name="light_grey"/>
-        </visual>
-        <collision>
-            <origin xyz="${gripper_finger_width/2} 0 -${gripper_finger_length/2}" rpy="0 0 0"/>
-            <geometry>
-                <box size="${gripper_finger_width} ${gripper_finger_height} ${gripper_finger_length}"/>
-            </geometry>
-        </collision>
-        <xacro:inertial_box mass="${gripper_finger_mass}" x="${gripper_finger_width}" y="${gripper_finger_height}" z="${gripper_finger_length}">
-            <origin xyz="${gripper_finger_width/2} 0 -${gripper_finger_length/2}" rpy="0 0 0"/>
-        </xacro:inertial_box>
-    </link>
-    <gazebo reference="right_gripper_finger1">
-        <material>Gazebo/Grey</material>
-    </gazebo>
-     <!-- +++++++++++++++++++++++++++++++++++++++++++++++++++++++++++++++++++++++++ -->
-     <!-- Right Gripper Finger 1 extension (fixed to finger1) -->
-    <joint name="right_gripper_finger1_ext_joint" type="fixed">
-        <parent link="right_gripper_finger1"/>
-        <child link="right_gripper_finger1_ext"/>
-        <origin xyz="${gripper_palm_width/128} 0 -${gripper_palm_length*1.15}" rpy="0 1.04 0"/>
-    </joint>
-    <link name="right_gripper_finger1_ext">
-        <visual>
-            <origin xyz="${gripper_finger_width/2} 0 -${gripper_finger_length/2}" rpy="0 0 0"/>
-            <geometry>
-                <box size="${gripper_finger_ext_width} ${gripper_finger_ext_height} ${gripper_finger_ext_length}"/>
-            </geometry>
-            <material name="light_grey"/>
-        </visual>
-        <collision>
-            <origin xyz="${gripper_finger_ext_width/2} 0 -${gripper_finger_ext_length/2}" rpy="0 0 0"/>
-            <geometry>
-                <box size="${gripper_finger_ext_width} ${gripper_finger_ext_height} ${gripper_finger_ext_length}"/>
-            </geometry>
-        </collision>
-        <xacro:inertial_box mass="${gripper_finger_ext_mass}" x="${gripper_finger_ext_width}" y="${gripper_finger_ext_height}" z="${gripper_finger_ext_length}">
-            <origin xyz="${gripper_finger_ext_width/2} 0 -${gripper_finger_ext_length/2}" rpy="0 0 0"/>
-        </xacro:inertial_box>
-    </link>
-    <gazebo reference="right_gripper_finger1_ext">
-        <material>Gazebo/Grey</material>
-    </gazebo>
-    <!-- +++++++++++++++++++++++++++++++++++++++++++++++++++++++++++++++++++++++++ -->
-    <!-- Right Gripper Finger 2 (revolute, same shape as finger1, mirrored) -->
-    <joint name="right_gripper_finger2_joint" type="revolute">
-        <parent link="right_gripper_palm"/>
-        <child link="right_gripper_finger2"/>
         <origin xyz="-${gripper_palm_width/8} 0.019 -${gripper_palm_length/1.75}" rpy=".0325 0.925 0"/>
         <axis xyz="0 -1 0"/>
@@ -292,4 +292,50 @@
         <dynamics damping="0.2" friction="0.05"/>
     </joint>
+    <link name="right_gripper_finger1">
+        <collision>
+            <origin xyz="-${gripper_finger_width/2} 0 -${gripper_finger_length/2}" rpy="0 0 0"/>
+            <geometry>
+                <box size="${gripper_finger_width} ${gripper_finger_height} ${gripper_finger_length}"/>
+            </geometry>
+        </collision>
+        <xacro:inertial_box mass="${gripper_finger_mass}" x="${gripper_finger_width}" y="${gripper_finger_height}" z="${gripper_finger_length}">
+            <origin xyz="-${gripper_finger_width/2} 0 -${gripper_finger_length/2}" rpy="0 0 0"/>
+        </xacro:inertial_box>
+    </link>
+    <gazebo reference="right_gripper_finger1">
+        <material>Gazebo/Grey</material>
+    </gazebo>
+    <!-- +++++++++++++++++++++++++++++++++++++++++++++++++++++++++++++++++++++++++ -->
+    <!-- Right Gripper Finger 2 extension (fixed to finger2) -->
+    <joint name="right_gripper_finger1_ext_joint" type="fixed">
+        <parent link="right_gripper_finger1"/>
+        <child link="right_gripper_finger1_ext"/>
+        <origin xyz=".01 0 -${gripper_palm_length}" rpy="0 -.965 0"/>
+    </joint>
+    <link name="right_gripper_finger1_ext">
+        <collision>
+            <origin xyz="-${gripper_finger_ext_width/2} 0 -${gripper_finger_ext_length/3.5}" rpy="0 0 0"/>
+            <geometry>
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