Commit message: refactor: reconfigure gripper kinematics by updating joint naming and URDF structures

File: src/nav/bonicbot_a2_description/urdf/ros2_control.xacro (robot description, xacro)
@@ -53,5 +53,18 @@
       </joint>
       <!-- Grippers - Primary fingers -->
+      <joint name="left_gripper_finger1_joint">
+        <command_interface name="position"/>
+        <state_interface name="position"/>
+        <state_interface name="velocity"/>
+      </joint>
+      <joint name="right_gripper_finger1_joint">
+        <command_interface name="position"/>
+        <state_interface name="position"/>
+        <state_interface name="velocity"/>
+      </joint>
+      <!-- Grippers - Mimic fingers -->
       <joint name="left_gripper_finger2_joint">
+        <param name="mimic">left_gripper_finger1_joint</param>
+        <param name="multiplier">1</param>
         <command_interface name="position"/>
         <state_interface name="position"/>
@@ -59,18 +72,5 @@
       </joint>
       <joint name="right_gripper_finger2_joint">
-        <command_interface name="position"/>
-        <state_interface name="position"/>
-        <state_interface name="velocity"/>
-      </joint>
-      <!-- Grippers - Mimic fingers -->
-      <joint name="left_gripper_finger3_joint">
-        <param name="mimic">left_gripper_finger2_joint</param>
-        <param name="multiplier">1</param>
-        <command_interface name="position"/>
-        <state_interface name="position"/>
-        <state_interface name="velocity"/>
-      </joint>
-      <joint name="right_gripper_finger3_joint">
-        <param name="mimic">right_gripper_finger2_joint</param>
+        <param name="mimic">right_gripper_finger1_joint</param>
         <param name="multiplier">1</param>
         <command_interface name="position"/>
@@ -152,5 +152,5 @@
       </joint>
       <!-- Grippers - Primary fingers -->
-      <joint name="left_gripper_finger2_joint">
+      <joint name="left_gripper_finger1_joint">
         <command_interface name="position"/>
         <param name="min">-0.785</param>  <!-- -45 degrees -->
@@ -159,5 +159,5 @@
         <state_interface name="velocity"/>
       </joint>
-      <joint name="right_gripper_finger2_joint">
+      <joint name="right_gripper_finger1_joint">
         <command_interface name="position"/>
         <param name="min">-0.785</param>  <!-- -45 degrees -->

Commit message: fix: invert gripper joint limits and update documentation to reflect driven finger numbering alignment with M1

File: src/nav/bonicbot_a2_description/urdf/gripper.xacro (robot description, xacro)
@@ -148,5 +148,5 @@
         <origin xyz="-${gripper_palm_width/8} 0.011 -${gripper_palm_length/1.75}" rpy="-.0325 0.925 0"/>
         <axis xyz="0 -1 0"/>
-        <limit lower="-1.047" upper="0.785" effort="10.0" velocity="5.0"/>
+        <limit lower="-0.785" upper="1.047" effort="10.0" velocity="5.0"/>
         <dynamics damping="0.0" friction="0.0"/>
         <mimic joint="left_gripper_finger1_joint" multiplier="1"/>
@@ -334,5 +334,5 @@
         <origin xyz="-${gripper_palm_width/8} 0.041 -${gripper_palm_length/1.75}" rpy=".0325 0.925 0"/>
         <axis xyz="0 -1 0"/>
-        <limit lower="-1.047" upper="0.785" effort="10.0" velocity="5.0"/>
+        <limit lower="-0.785" upper="1.047" effort="10.0" velocity="5.0"/>
         <dynamics damping="0.0" friction="0.0"/>
         <mimic joint="right_gripper_finger1_joint" multiplier="1"/>
