Commit message: fix: correct elbow joint limits in kinematic URDF to -50..0 deg
body.xacro had the same inverted range as the ros2_control block fixed
in db94ea1 (0..50 instead of -50..0), duplicated for both left and
right elbow. This is the limit robot_state_publisher and ros2_control's
joint-limit enforcement actually read from, so the earlier fix alone
wasn't enough — negative elbow commands were still being clamped to 0.

File: src/nav/bonicbot_a2_description/urdf/body.xacro (robot description, xacro)
@@ -157,5 +157,5 @@
         <origin xyz="0 0 -${upper_arm_length/2}" rpy="-0.235 0 0"/>
         <axis xyz="0 -0.9725 -0.2328"/>
-        <limit lower="0" upper="0.873" effort="5.0" velocity="2.0"/>
+        <limit lower="-0.873" upper="0" effort="5.0" velocity="2.0"/>
         <dynamics damping="0.5" friction="0.1"/>
     </joint>
@@ -279,5 +279,5 @@
         <origin xyz="0 0 -${upper_arm_length/2}" rpy="0.235 0 0"/>
         <axis xyz="0 -0.9725 0.2328"/>
-        <limit lower="0" upper="0.873" effort="5.0" velocity="2.0"/>
+        <limit lower="-0.873" upper="0" effort="5.0" velocity="2.0"/>
         <dynamics damping="0.5" friction="0.1"/>
     </joint>

Commit message: fix: reverse elbow joint axes for visual alignment and update navigation parameters to respect hardware velocity and acceleration limits

File: src/nav/bonicbot_a2_description/urdf/body.xacro (robot description, xacro)
@@ -156,5 +156,15 @@
         <child link="left_forearm"/>
         <origin xyz="0 0 -${upper_arm_length/2}" rpy="-0.235 0 0"/>
-        <axis xyz="0 -0.9725 -0.2328"/>
+        <!-- Axis reversed 2026-08-25: the physical elbow moved correctly for a
+             given command while RViz rendered its mirror image, on the SAME
+             /joint_states sample — an objective URDF-vs-hardware disagreement,
+             not a matter of expectation. Gazebo agreed with RViz because both
+             read this file. Fixed here rather than by re-adding elbow IDs
+             (4, 11) to isServoInverted(), which would have made RViz match by
+             breaking the real arm.
+             Reversing the axis vector alone mirrors the motion while leaving
+             the limits (and therefore the -0.873..0 command convention that
+             the registry, firmware and robot_app all share) untouched. -->
+        <axis xyz="0 0.9725 0.2328"/>
         <limit lower="-0.873" upper="0" effort="5.0" velocity="2.0"/>
         <dynamics damping="0.5" friction="0.1"/>
@@ -278,5 +288,15 @@
         <child link="right_forearm"/>
         <origin xyz="0 0 -${upper_arm_length/2}" rpy="0.235 0 0"/>
-        <axis xyz="0 -0.9725 0.2328"/>
+        <!-- Axis reversed 2026-08-25: the physical elbow moved correctly for a
+             given command while RViz rendered its mirror image, on the SAME
+             /joint_states sample — an objective URDF-vs-hardware disagreement,
+             not a matter of expectation. Gazebo agreed with RViz because both
+             read this file. Fixed here rather than by re-adding elbow IDs
+             (4, 11) to isServoInverted(), which would have made RViz match by
+             breaking the real arm.
+             Reversing the axis vector alone mirrors the motion while leaving
+             the limits (and therefore the -0.873..0 command convention that
+             the registry, firmware and robot_app all share) untouched. -->
+        <axis xyz="0 0.9725 -0.2328"/>
         <limit lower="-0.873" upper="0" effort="5.0" velocity="2.0"/>
         <dynamics damping="0.5" friction="0.1"/>
