Commit message: fix: update docking camera position and tune docking configuration parameters

File: src/nav/bonicbot_a2_description/urdf/docking_camera.xacro (robot description, xacro)
@@ -44,5 +44,32 @@
              because the robot reverses onto the dock (docking.yaml
              dock_backwards: true). -->
-        <origin xyz="-0.110 0 0.120" rpy="0 0 ${pi}"/>
+        <!-- x=-0.180: THE LENS MUST SIT OUTSIDE THE ROBOT'S OWN GEOMETRY.
+             There are TWO nested enclosures here and both have to be cleared:
+               chassis box   ends at x = -0.114  (chassis_length 0.228 / 2)
+               body.obj shell ends at x = -0.1396 AT THIS CAMERA'S HEIGHT
+                                                  (measured from the mesh's own
+                                                   vertices within z +/-0.02 of
+                                                   0.120; the shell's overall
+                                                   bbox reaches -0.157, but that
+                                                   is a different part of the
+                                                   shell, not at this height)
+             The original -0.110 was inside BOTH. A first fix to -0.135 cleared
+             the chassis box but was still inside the shell, which is why the
+             camera then rendered perfectly while stationary and at staging
+             (0 blanks over 47 frames) yet broke up as soon as the robot moved
+             and rotated: the surrounding shell triangles fall in and out of
+             the 0.05m near-clip as the pose changes, and a frame that clips
+             wrong comes out a single flat colour with no scene at all.
+             face_camera never shows this because it sits on the head at
+             z~0.685, above the shell, enclosed by nothing.
+             Diagnosed 2026-09-23 by logging both cameras over 2.2m of travel:
+             face 394-601 unique colours throughout, docking exactly 1.
+             -0.155 clears the shell by 15mm at this height. That also matches
+             what the real addon is: a bracket bolted to the BACK of the robot,
+             so the lens genuinely does protrude past the shell.
+             DO NOT move it forward of about -0.145. Re-measure on the real
+             mount, and if you change the height, re-run the vertex query above
+             for the new z first; the shell's rear extent varies with z. -->
+        <origin xyz="-0.155 0 0.120" rpy="0 0 ${pi}"/>
     </joint>
     <!-- Prevent URDF→SDF fixed-joint reduction from lumping this link into
@@ -104,5 +131,5 @@
         <sensor name="docking_camera" type="camera">
             <pose> 0 0 0 0 0 0 </pose>
-            <visualize>false</visualize>
+            <visualize>true</visualize>  <!-- TEMP debug 2026-09-23: watch the frustum/preview live while chasing the blank-on-yaw bug -->
             <update_rate>10</update_rate>
             <camera>

File: src/nav/bonicbot_a2_description/urdf/robot_core.xacro (robot description, xacro)
@@ -109,4 +109,17 @@
         <origin xyz="${-wheel_offset_x} 0 ${-wheel_offset_z}"/>
     </joint>
+    <!-- TRIED disableFixedJointLumping on chassis_joint (2026-09-23), on the
+         theory that docking_camera's blank-during-yaw bug traced to chassis
+         being the one unlumped-camera-mount link without it. WRONG — it broke
+         model spawn entirely:
+             PoseRelativeToGraph unable to find path to source vertex
+         Reverted. The docking-camera-blank-on-yaw bug is CONFIRMED (see
+         docking.yaml and docs/bonicbot_a2_docking.md) but the fix is not this.
+         Something else about chassis's role in the pose graph makes it load
+         bearing for lumping to stay enabled here — chassis carries several
+         children (laser_joint, wheel joints reference base_link not chassis,
+         but body/external mesh and lidar do reference it) and disabling
+         lumping on it alone, without matching changes elsewhere, produces an
+         inconsistent graph rather than a fixed one. -->
     <link name="chassis">
         <visual>
